File: Hardware/PP-Rev2.sch (EAGLE design)
At the start: 182 parts, among them IC1 LT6004, IC2 TLC6C5912-Q1, Q1 MOSFET-PCHANNEL, Q10 2N7002PW, Q11 2N7002PW, Q12 2N7002PW, Q13 2N7002PW, Q14 2N7002PW, Q15 2N7002PW, Q2 MOSFET-PCHANNEL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

Commit message: additional work on board layout. Changed charger input terminals from bolt holes to large screw terminal
Parts:
- removed CHARGER+, CHARGER-: TERMINAL_HOLE, MRDT-2015-PowerBoard:TERMINAL_HOLE
- added J1: J_0399700102, MRDT-2014-All:J_0399700102
Connections:
- net CHARGER+: now also J1.1-1, J1.1-2; no longer CHARGER+.P$1
- net GND: now also J1.2-1, J1.2-2; no longer CHARGER-.P$1
Changed lines of the file:
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@@
 <?xml version="1.0" encoding="utf-8"?>
 <!DOCTYPE eagle SYSTEM "eagle.dtd">
-<eagle version="7.1.0">
+<eagle version="6.5.0">
 <drawing>
 <settings>
@@
 <setting verticaltext="up"/>
 </settings>
-<grid distance="0.1" unitdist="inch" unit="inch" style="lines" multiple="1" display="no" altdistance="0.01" altunitdist="inch" altunit="inch"/>
+<grid distance="0.1" unitdist="inch" unit="inch" style="lines" multiple="1" display="yes" altdistance="0.01" altunitdist="inch" altunit="inch"/>
 <layers>
 <layer number="1" name="Top" color="4" fill="1" visible="no" active="no"/>
+<layer number="2" name="Route2" color="1" fill="3" visible="no" active="no"/>
+<layer number="3" name="Route3" color="4" fill="3" visible="no" active="no"/>
+<layer number="4" name="Route4" color="1" fill="4" visible="no" active="no"/>
+<layer number="5" name="Route5" color="4" fill="4" visible="no" active="no"/>
+<layer number="6" name="Route6" color="1" fill="8" visible="no" active="no"/>
+<layer number="7" name="Route7" color="4" fill="8" visible="no" active="no"/>
+<layer number="8" name="Route8" color="1" fill="2" visible="no" active="no"/>
+<layer number="9" name="Route9" color="4" fill="2" visible="no" active="no"/>
+<layer number="10" name="Route10" color="1" fill="7" visible="no" active="no"/>
+<layer number="11" name="Route11" color="4" fill="7" visible="no" active="no"/>
+<layer number="12" name="Route12" color="1" fill="5" visible="no" active="no"/>
+<layer number="13" name="Route13" color="4" fill="5" visible="no" active="no"/>
+<layer number="14" name="Route14" color="1" fill="6" visible="no" active="no"/>
+<layer number="15" name="Route15" color="4" fill="6" visible="no" active="no"/>
 <layer number="16" name="Bottom" color="1" fill="1" visible="no" active="no"/>
 <layer number="17" name="Pads" color="2" fill="1" visible="no" active="no"/>
@@
 <part name="GND28" library="SparkFun-Aesthetics" deviceset="GND" device=""/>
 <part name="U$12" library="2016PowerPackLibraries" deviceset="LTC4440" device=""/>
-<part name="CHARGER+" library="MRDT-2015-PowerBoard" deviceset="TERMINAL_HOLE" device=""/>
-<part name="CHARGER-" library="MRDT-2015-PowerBoard" deviceset="TERMINAL_HOLE" device=""/>
 <part name="R43" library="resistor" deviceset="R-US_" device="R1206" value="100kΩ"/>
 <part name="R44" library="resistor" deviceset="R-US_" device="R1206" value="10kΩ"/>
@@
 <part name="U$15" library="MAX3077" deviceset="MAX3077" device=""/>
 <part name="P+10" library="supply1" deviceset="+5V" device=""/>
+<part name="J1" library="MRDT-2014-All" deviceset="J_0399700102" device=""/>
 </parts>
 <sheets>
@@
 <instance part="GND28" gate="1" x="50.8" y="307.34"/>
 <instance part="U$12" gate="G$1" x="-35.56" y="279.4"/>
-<instance part="CHARGER+" gate="G$1" x="68.58" y="327.66"/>
-<instance part="CHARGER-" gate="G$1" x="86.36" y="327.66"/>
 <instance part="R43" gate="G$1" x="43.18" y="335.28" rot="R270"/>
 <instance part="R44" gate="G$1" x="43.18" y="350.52" rot="R270"/>
@@
 <instance part="U$15" gate="G$1" x="454.66" y="269.24" rot="R180"/>
 <instance part="P+10" gate="1" x="449.58" y="256.54"/>
+<instance part="J1" gate="G$1" x="76.2" y="337.82" rot="R90"/>
 </instances>
 <busses>
@@
 <junction x="50.8" y="312.42"/>
 <pinref part="GND28" gate="1" pin="GND"/>
-<pinref part="CHARGER-" gate="G$1" pin="P$1"/>
 <wire x1="86.36" y1="327.66" x2="86.36" y2="312.42" width="0.1524" layer="91"/>
 <wire x1="86.36" y1="312.42" x2="55.88" y2="312.42" width="0.1524" layer="91"/>
 <junction x="55.88" y="312.42"/>
+<pinref part="J1" gate="G$1" pin="2-1"/>
+<wire x1="78.74" y1="330.2" x2="78.74" y2="327.66" width="0.1524" layer="91"/>
+<wire x1="78.74" y1="327.66" x2="81.28" y2="327.66" width="0.1524" layer="91"/>
+<pinref part="J1" gate="G$1" pin="2-2"/>
+<wire x1="81.28" y1="327.66" x2="86.36" y2="327.66" width="0.1524" layer="91"/>
+<wire x1="81.28" y1="330.2" x2="81.28" y2="327.66" width="0.1524" layer="91"/>
+<junction x="81.28" y="327.66"/>
 </segment>
 <segment>
@@
 <wire x1="55.88" y1="325.12" x2="55.88" y2="322.58" width="0.1524" layer="91"/>
 <junction x="45.72" y="325.12"/>
-<pinref part="CHARGER+" gate="G$1" pin="P$1"/>
 <wire x1="55.88" y1="325.12" x2="68.58" y2="325.12" width="0.1524" layer="91"/>
 <wire x1="68.58" y1="325.12" x2="68.58" y2="327.66" width="0.1524" layer="91"/>
@@
 <junction x="43.18" y="325.12"/>
 <label x="58.42" y="325.12" size="1.778" layer="95"/>
-</segment>
-<segment>
+<pinref part="J1" gate="G$1" pin="1-1"/>
+<wire x1="73.66" y1="330.2" x2="73.66" y2="327.66" width="0.1524" layer="91"/>
+<wire x1="73.66" y1="327.66" x2="71.12" y2="327.66" width="0.1524" layer="91"/>
+<pinref part="J1" gate="G$1" pin="1-2"/>
+<wire x1="71.12" y1="327.66" x2="68.58" y2="327.66" width="0.1524" layer="91"/>
+<wire x1="71.12" y1="330.2" x2="71.12" y2="327.66" width="0.1524" layer="91"/>
+<junction x="71.12" y="327.66"/>
+</segment>
+<segment>

Commit message: Lots of power supply routing. Merged two independent 5V supplies into one supply
Connections:
- removed net +5V: C22.1, U$15.VCC, U$2.VCC, U$4.VCC
- net 5V: now also C22.1, U$15.VCC, U$2.VCC, U$4.VCC
Other:
- moved on the sheet: C22
Changed lines of the file:
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@@
 <part name="GND20" library="supply1" deviceset="GND" device=""/>
 <part name="U$2" library="MRDT-2015-BMS" deviceset="ACS770" device=""/>
-<part name="P+1" library="supply1" deviceset="+5V" device=""/>
 <part name="GND21" library="supply1" deviceset="GND" device=""/>
 <part name="V_ARRAY" library="MRDT-2015-PowerBoard" deviceset="TERMINAL_HOLE" device=""/>
@@
 <part name="U$4" library="MRDT-2015-BMS" deviceset="ACS770" device=""/>
 <part name="GND29" library="supply1" deviceset="GND" device=""/>
-<part name="P+2" library="supply1" deviceset="+5V" device=""/>
 <part name="U$5" library="2016PowerPackLibraries" deviceset="AGP4233" device="" value="AGP4233-223ME"/>
 <part name="U$3" library="MRDT-2015-PowerBoard" deviceset="C_108CKH050M" device=""/>
@@
 <part name="R73" library="SparkFun-Passives" deviceset="RESISTOR" device="1206" value="120 Ohm"/>
 <part name="GND54" library="SparkFun-Aesthetics" deviceset="GND" device=""/>
-<part name="P+9" library="supply1" deviceset="+5V" device=""/>
 <part name="GND55" library="SparkFun-Aesthetics" deviceset="GND" device=""/>
 <part name="GND56" library="SparkFun-Aesthetics" deviceset="GND" device=""/>
 <part name="C22" library="resistor" deviceset="C-US" device="C1206" value="1uF"/>
 <part name="U$15" library="MAX3077" deviceset="MAX3077" device=""/>
-<part name="P+10" library="supply1" deviceset="+5V" device=""/>
 <part name="J1" library="MRDT-2014-All" deviceset="J_0399700102" device=""/>
+<part name="SUPPLY12" library="SparkFun-Aesthetics" deviceset="5V" device=""/>
+<part name="SUPPLY13" library="SparkFun-Aesthetics" deviceset="5V" device=""/>
+<part name="SUPPLY14" library="SparkFun-Aesthetics" deviceset="5V" device=""/>
 </parts>
 <sheets>
@@
 <instance part="GND20" gate="1" x="-12.7" y="25.4"/>
 <instance part="U$2" gate="G$1" x="-93.98" y="223.52" rot="R90"/>
-<instance part="P+1" gate="1" x="-91.44" y="248.92"/>
 <instance part="GND21" gate="1" x="-101.6" y="241.3"/>
 <instance part="V_ARRAY" gate="G$1" x="-116.84" y="213.36"/>
@@
 <instance part="U$4" gate="G$1" x="-63.5" y="335.28" rot="R90"/>
 <instance part="GND29" gate="1" x="-73.66" y="363.22"/>
-<instance part="P+2" gate="1" x="-60.96" y="375.92"/>
 <instance part="U$5" gate="G$1" x="-7.62" y="325.12" rot="R90"/>
 <instance part="U$3" gate="G$1" x="-25.4" y="317.5" smashed="yes">
@@
 <instance part="R73" gate="G$1" x="434.34" y="274.32"/>
 <instance part="GND54" gate="1" x="480.06" y="276.86"/>
-<instance part="P+9" gate="1" x="480.06" y="261.62"/>
 <instance part="GND55" gate="1" x="421.64" y="281.94"/>
-<instance part="GND56" gate="1" x="449.58" y="238.76"/>
-<instance part="C22" gate="G$1" x="449.58" y="248.92"/>
+<instance part="GND56" gate="1" x="472.44" y="246.38"/>
+<instance part="C22" gate="G$1" x="472.44" y="256.54"/>
 <instance part="U$15" gate="G$1" x="454.66" y="269.24" rot="R180"/>
-<instance part="P+10" gate="1" x="449.58" y="256.54"/>
 <instance part="J1" gate="G$1" x="76.2" y="337.82" rot="R90"/>
+<instance part="SUPPLY12" gate="G$1" x="474.98" y="261.62"/>
+<instance part="SUPPLY13" gate="G$1" x="-91.44" y="241.3"/>
+<instance part="SUPPLY14" gate="G$1" x="-60.96" y="353.06"/>
 </instances>
 <busses>
@@
 </segment>
 <segment>
+<pinref part="C22" gate="G$1" pin="2"/>
 <pinref part="GND56" gate="1" pin="GND"/>
-<wire x1="449.58" y1="241.3" x2="449.58" y2="243.84" width="0.1524" layer="91"/>
-<pinref part="C22" gate="G$1" pin="2"/>
+<wire x1="472.44" y1="251.46" x2="472.44" y2="248.92" width="0.1524" layer="91"/>
 </segment>
 </net>
@@
 <wire x1="-12.7" y1="38.1" x2="-2.54" y2="38.1" width="0.1524" layer="91"/>
 <junction x="-12.7" y="38.1"/>
-</segment>
-</net>
-<net name="+5V" class="0">
-<segment>
-<pinref part="P+1" gate="1" pin="+5V"/>
-<pinref part="U$2" gate="G$1" pin="VCC"/>
-<wire x1="-91.44" y1="246.38" x2="-91.44" y2="236.22" width="0.1524" layer="91"/>
-</segment>
-<segment>
-<pinref part="U$4" gate="G$1" pin="VCC"/>
-<pinref part="P+2" gate="1" pin="+5V"/>
-<wire x1="-60.96" y1="347.98" x2="-60.96" y2="373.38" width="0.1524" layer="91"/>
-</segment>
-<segment>
-<wire x1="469.9" y1="261.62" x2="474.98" y2="261.62" width="0.1524" layer="91"/>
-<wire x1="474.98" y1="261.62" x2="474.98" y2="256.54" width="0.1524" layer="91"/>
-<pinref part="P+9" gate="1" pin="+5V"/>
-<wire x1="474.98" y1="256.54" x2="480.06" y2="256.54" width="0.1524" layer="91"/>
-<wire x1="480.06" y1="256.54" x2="480.06" y2="259.08" width="0.1524" layer="91"/>
-<pinref part="U$15" gate="G$1" pin="VCC"/>
-</segment>
-<segment>
-<pinref part="C22" gate="G$1" pin="1"/>
-<pinref part="P+10" gate="1" pin="+5V"/>
-<wire x1="449.58" y1="251.46" x2="449.58" y2="254" width="0.1524" layer="91"/>
 </segment>
 </net>
@@
 <wire x1="467.36" y1="170.18" x2="467.36" y2="167.64" width="0.1524" layer="91"/>
 </segment>
-</net>
+<segment>
+<pinref part="U$15" gate="G$1" pin="VCC"/>
+<pinref part="SUPPLY12" gate="G$1" pin="5V"/>
+<wire x1="469.9" y1="261.62" x2="472.44" y2="261.62" width="0.1524" layer="91"/>
+<pinref part="C22" gate="G$1" pin="1"/>
+<wire x1="472.44" y1="261.62" x2="474.98" y2="261.62" width="0.1524" layer="91"/>
+<wire x1="472.44" y1="261.62" x2="472.44" y2="259.08" width="0.1524" layer="91"/>
+<junction x="472.44" y="261.62"/>
+</segment>
+<segment>
+<pinref part="SUPPLY14" gate="G$1" pin="5V"/>
+<pinref part="U$4" gate="G$1" pin="VCC"/>
+<wire x1="-60.96" y1="353.06" x2="-60.96" y2="347.98" width="0.1524" layer="91"/>
+</segment>
+<segment>
+<pinref part="SUPPLY13" gate="G$1" pin="5V"/>
+<pinref part="U$2" gate="G$1" pin="VCC"/>
+<wire x1="-91.44" y1="241.3" x2="-91.44" y2="236.22" width="0.1524" layer="91"/>
+</segment>
+</net>
