File: Hardware/Main-BMS/BMS.sch (EAGLE design)
At the start: 141 parts, among them IC1 ACS759, IC2 TLC6C5912-Q1, J3 APPPP45_PCB_VERT, Q1 2N7002PW, Q11 2N7002PW, Q12 2N7002PW, Q13 2N7002PW, Q14 2N7002PW, Q15 2N7002PW, Q2 2N7002PW, Q3 2N7002PW, U2 MAX232, X5 22-23-2041

Commit message: Tidying up and part swap
Rounded dimensions 5"x5.2", rearranged labels, updated connectors to
sync with MRDT-Connectors, rearranged vias.
Changed out MAX232 (5V operation) for MAX3232 (3V to 5V)
Parts:
- C44, C45, C46, C47, C48: value 1u -> 0.1u
- U2: value MAX232 -> MAX3232D; device MRDT-ICs:MAX232 -> MRDT-ICs:MAX3232D
- renumbered IRLS3034-7P to Q17, IRLS3034-7P1 to Q16
Connections:
- net +3V3: now also C46.1, U2.VCC
- net 5V: no longer C46.1, U2.VCC
- net GND: now also RS232_IND.1, RS232_PB.1; no longer RS232_IND.2, RS232_PB.2
- net RS232_TX_IND: now also RS232_IND.2; no longer RS232_IND.1
- net RS232_TX_PB: now also RS232_PB.2; no longer RS232_PB.1
Changed lines of the file:
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@@
 <part name="GND21" library="supply1" deviceset="GND" device=""/>
 <part name="V_IN" library="MRDT-2015-PowerBoard" deviceset="TERMINAL_HOLE" device=""/>
-<part name="IRLS3034-7P" library="MRDT-2015-BMS" deviceset="IRLS3034-7P" device=""/>
+<part name="Q17" library="MRDT-2015-BMS" deviceset="IRLS3034-7P" device=""/>
 <part name="V_OUT" library="MRDT-2015-PowerBoard" deviceset="TERMINAL_HOLE" device=""/>
 <part name="R38" library="resistor" deviceset="R-US_" device="R1206" value="100kΩ"/>
@@
 <part name="R19" library="rcl" deviceset="R-US_" device="R0603" value="1M"/>
 <part name="R21" library="rcl" deviceset="R-US_" device="R0603" value="1M"/>
-<part name="IRLS3034-7P1" library="MRDT-2015-BMS" deviceset="IRLS3034-7P" device=""/>
+<part name="Q16" library="MRDT-2015-BMS" deviceset="IRLS3034-7P" device=""/>
 <part name="+3V3" library="supply1" deviceset="+3V3" device=""/>
 <part name="SUPPLY6" library="SparkFun-Aesthetics" deviceset="5V" device=""/>
@@
 <part name="U$16" library="MRDT-Connectors" deviceset="SL02-VERT" device=""/>
 <part name="GND36" library="SparkFun-Aesthetics" deviceset="GND" device=""/>
-<part name="U2" library="MRDT-ICs" deviceset="MAX232" device=""/>
-<part name="C44" library="SparkFun-Passives" deviceset="CAP" device="0805" value="1u"/>
-<part name="C45" library="SparkFun-Passives" deviceset="CAP" device="0805" value="1u"/>
-<part name="C46" library="SparkFun-Passives" deviceset="CAP" device="0805" value="1u"/>
+<part name="U2" library="MRDT-ICs" deviceset="MAX*232" device="D" technology="3" value="MAX3232D"/>
+<part name="C44" library="SparkFun-Passives" deviceset="CAP" device="0805" value="0.1u"/>
+<part name="C45" library="SparkFun-Passives" deviceset="CAP" device="0805" value="0.1u"/>
+<part name="C46" library="SparkFun-Passives" deviceset="CAP" device="0805" value="0.1u"/>
 <part name="GND15" library="SparkFun-Aesthetics" deviceset="GND" device=""/>
 <part name="GND44" library="SparkFun-Aesthetics" deviceset="GND" device=""/>
-<part name="C47" library="SparkFun-Passives" deviceset="CAP" device="0805" value="1u"/>
-<part name="C48" library="SparkFun-Passives" deviceset="CAP" device="0805" value="1u"/>
+<part name="C47" library="SparkFun-Passives" deviceset="CAP" device="0805" value="0.1u"/>
+<part name="C48" library="SparkFun-Passives" deviceset="CAP" device="0805" value="0.1u"/>
 <part name="GND16" library="SparkFun-Aesthetics" deviceset="GND" device=""/>
 <part name="GND17" library="SparkFun-Aesthetics" deviceset="GND" device=""/>
-<part name="SUPPLY14" library="SparkFun-Aesthetics" deviceset="5V" device=""/>
 <part name="RS232_IND" library="MRDT-Connectors" deviceset="SL03" device=""/>
 <part name="RS232_PB" library="MRDT-Connectors" deviceset="SL03" device=""/>
 <part name="GND18" library="SparkFun-Aesthetics" deviceset="GND" device=""/>
+<part name="+3V7" library="supply1" deviceset="+3V3" device=""/>
 </parts>
 <sheets>
@@
 <instance part="GND21" gate="1" x="43.18" y="-101.6" rot="MR0"/>
 <instance part="V_IN" gate="G$1" x="25.4" y="-66.04" rot="MR0"/>
-<instance part="IRLS3034-7P" gate="G$1" x="134.62" y="-78.74" rot="R90"/>
+<instance part="Q17" gate="G$1" x="134.62" y="-78.74" rot="R90"/>
 <instance part="V_OUT" gate="G$1" x="220.98" y="-66.04"/>
 <instance part="R38" gate="G$1" x="177.8" y="-81.28" rot="R270"/>
@@
 <instance part="R19" gate="G$1" x="220.98" y="-162.56" rot="R180"/>
 <instance part="R21" gate="G$1" x="220.98" y="-167.64" rot="R180"/>
-<instance part="IRLS3034-7P1" gate="G$1" x="160.02" y="-55.88" rot="R90"/>
+<instance part="Q16" gate="G$1" x="160.02" y="-55.88" rot="R90"/>
 <instance part="+3V3" gate="G$1" x="607.06" y="-187.96"/>
 <instance part="SUPPLY6" gate="G$1" x="502.92" y="-152.4"/>
@@
 <instance part="GND16" gate="1" x="553.72" y="-83.82"/>
 <instance part="GND17" gate="1" x="553.72" y="-91.44"/>
-<instance part="SUPPLY14" gate="G$1" x="528.32" y="-53.34"/>
 <instance part="RS232_IND" gate="G$1" x="607.06" y="-116.84"/>
 <instance part="RS232_PB" gate="G$1" x="607.06" y="-96.52"/>
 <instance part="GND18" gate="1" x="594.36" y="-104.14"/>
+<instance part="+3V7" gate="G$1" x="528.32" y="-55.88"/>
 </instances>
 <busses>
@@
 </segment>
 <segment>
+<pinref part="RS232_PB" gate="G$1" pin="1"/>
 <pinref part="GND18" gate="1" pin="GND"/>
-<wire x1="594.36" y1="-101.6" x2="594.36" y2="-96.52" width="0.1524" layer="91"/>
-<pinref part="RS232_PB" gate="G$1" pin="2"/>
-<wire x1="594.36" y1="-96.52" x2="599.44" y2="-96.52" width="0.1524" layer="91"/>
-</segment>
-<segment>
+<wire x1="599.44" y1="-99.06" x2="594.36" y2="-99.06" width="0.1524" layer="91"/>
+<wire x1="594.36" y1="-99.06" x2="594.36" y2="-101.6" width="0.1524" layer="91"/>
+</segment>
+<segment>
+<pinref part="RS232_IND" gate="G$1" pin="1"/>
 <pinref part="GND36" gate="1" pin="GND"/>
-<wire x1="594.36" y1="-121.92" x2="594.36" y2="-116.84" width="0.1524" layer="91"/>
-<pinref part="RS232_IND" gate="G$1" pin="2"/>
-<wire x1="594.36" y1="-116.84" x2="599.44" y2="-116.84" width="0.1524" layer="91"/>
+<wire x1="599.44" y1="-119.38" x2="594.36" y2="-119.38" width="0.1524" layer="91"/>
+<wire x1="594.36" y1="-119.38" x2="594.36" y2="-121.92" width="0.1524" layer="91"/>
 </segment>
 </net>
@@
 <net name="N$34" class="0">
 <segment>
-<pinref part="IRLS3034-7P" gate="G$1" pin="GATE"/>
+<pinref part="Q17" gate="G$1" pin="GATE"/>
 <wire x1="139.7" y1="-104.14" x2="139.7" y2="-91.44" width="0.1524" layer="91"/>
 <pinref part="ESTOP_1" gate="G$1" pin="1"/>
@@
 <wire x1="144.78" y1="-104.14" x2="139.7" y2="-104.14" width="0.1524" layer="91"/>
 <junction x="139.7" y="-104.14"/>
-<pinref part="IRLS3034-7P1" gate="G$1" pin="GATE"/>
+<pinref part="Q16" gate="G$1" pin="GATE"/>
 <wire x1="165.1" y1="-66.04" x2="154.94" y2="-66.04" width="0.1524" layer="91"/>
 <wire x1="154.94" y1="-66.04" x2="154.94" y2="-91.44" width="0.1524" layer="91"/>
@@
 <wire x1="124.46" y1="-17.78" x2="111.76" y2="-17.78" width="0.1524" layer="91"/>
 </segment>
-<segment>
-<pinref part="U2" gate="G$1" pin="VCC"/>
-<pinref part="SUPPLY14" gate="G$1" pin="5V"/>
-<wire x1="528.32" y1="-68.58" x2="528.32" y2="-60.96" width="0.1524" layer="91"/>
-<pinref part="C46" gate="G$1" pin="1"/>
-<wire x1="528.32" y1="-60.96" x2="528.32" y2="-53.34" width="0.1524" layer="91"/>
-<wire x1="500.38" y1="-60.96" x2="500.38" y2="-63.5" width="0.1524" layer="91"/>
-<wire x1="500.38" y1="-60.96" x2="528.32" y2="-60.96" width="0.1524" layer="91"/>
-<junction x="528.32" y="-60.96"/>
-</segment>
 </net>
 <net name="LOGIC_POWER" class="0">
@@
 <junction x="119.38" y="-81.28"/>
 <junction x="114.3" y="-76.2"/>
-<pinref part="IRLS3034-7P" gate="G$1" pin="DRAIN"/>
+<pinref part="Q17" gate="G$1" pin="DRAIN"/>
 <wire x1="127" y1="-76.2" x2="124.46" y2="-76.2" width="0.1524" layer="91"/>
 <junction x="119.38" y="-76.2"/>
@@
 <wire x1="124.46" y1="-76.2" x2="119.38" y2="-76.2" width="0.1524" layer="91"/>
 <wire x1="53.34" y1="-68.58" x2="53.34" y2="-76.2" width="0.1524" layer="91"/>
-<pinref part="IRLS3034-7P1" gate="G$1" pin="DRAIN"/>
+<pinref part="Q16" gate="G$1" pin="DRAIN"/>
 <wire x1="152.4" y1="-53.34" x2="124.46" y2="-53.34" width="0.1524" layer="91"/>
 <wire x1="124.46" y1="-53.34" x2="124.46" y2="-76.2" width="0.1524" layer="91"/>
@@
 <pinref part="IC1" gate="G$1" pin="VCC"/>
 </segment>
+<segment>
+<pinref part="U2" gate="G$1" pin="VCC"/>
+<pinref part="+3V7" gate="G$1" pin="+3V3"/>
+<wire x1="528.32" y1="-68.58" x2="528.32" y2="-63.5" width="0.1524" layer="91"/>
+<pinref part="C46" gate="G$1" pin="1"/>
+<wire x1="528.32" y1="-63.5" x2="528.32" y2="-58.42" width="0.1524" layer="91"/>
+<wire x1="500.38" y1="-63.5" x2="528.32" y2="-63.5" width="0.1524" layer="91"/>
+<junction x="528.32" y="-63.5"/>
+</segment>
 </net>
 <net name="CELL_1_BAL" class="0">
@@
 <segment>
 <pinref part="R38" gate="G$1" pin="1"/>
-<pinref part="IRLS3034-7P" gate="G$1" pin="SOURCE"/>
+<pinref part="Q17" gate="G$1" pin="SOURCE"/>
 <wire x1="177.8" y1="-76.2" x2="170.18" y2="-76.2" width="0.1524" layer="91"/>
-<pinref part="IRLS3034-7P1" gate="G$1" pin="SOURCE"/>
+<pinref part="Q16" gate="G$1" pin="SOURCE"/>
 <wire x1="170.18" y1="-76.2" x2="144.78" y2="-76.2" width="0.1524" layer="91"/>
 <wire x1="170.18" y1="-53.34" x2="170.18" y2="-76.2" width="0.1524" layer="91"/>
@@
 </segment>
 <segment>
-<label x="591.82" y="-99.06" size="1.27" layer="95" rot="R180" xref="yes"/>
-<pinref part="RS232_PB" gate="G$1" pin="1"/>
-<wire x1="591.82" y1="-99.06" x2="599.44" y2="-99.06" width="0.1524" layer="91"/>
+<label x="591.82" y="-96.52" size="1.27" layer="95" rot="R180" xref="yes"/>
+<pinref part="RS232_PB" gate="G$1" pin="2"/>
+<wire x1="599.44" y1="-96.52" x2="591.82" y2="-96.52" width="0.1524" layer="91"/>
 </segment>
 </net>
@@
 </segment>
 <segment>
-<label x="591.82" y="-119.38" size="1.27" layer="95" rot="R180" xref="yes"/>
-<pinref part="RS232_IND" gate="G$1" pin="1"/>
-<wire x1="591.82" y1="-119.38" x2="599.44" y2="-119.38" width="0.1524" layer="91"/>
-</segment>
-</net>
+<label x="591.82" y="-116.84" size="1.27" layer="95" rot="R180" xref="yes"/>
+<pinref part="RS232_IND" gate="G$1" pin="2"/>
+<wire x1="599.44" y1="-116.84" x2="591.82" y2="-116.84" width="0.1524" layer="91"/>
+</segment>
+</net>

Commit message: Indicator board connector
Added 5V pin to indicator board connector
Parts:
- removed RS232_IND: SL03, MRDT-Connectors:SL03
- added J1: SL04VERT, MRDT-Connectors:SL04VERT
- C46: value 0.1u -> 1u
Connections:
- net BUZZ_1 renamed BUZZER
- net 5V: now also J1.P$4
- net GND: now also J1.P$1; no longer RS232_IND.1
- net RS232_RX_IND: now also J1.P$3; no longer RS232_IND.3
- net RS232_TX_IND: now also J1.P$2; no longer RS232_IND.2
Changed lines of the file:
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@@
 <part name="C44" library="SparkFun-Passives" deviceset="CAP" device="0805" value="0.1u"/>
 <part name="C45" library="SparkFun-Passives" deviceset="CAP" device="0805" value="0.1u"/>
-<part name="C46" library="SparkFun-Passives" deviceset="CAP" device="0805" value="0.1u"/>
+<part name="C46" library="SparkFun-Passives" deviceset="CAP" device="0805" value="1u"/>
 <part name="GND15" library="SparkFun-Aesthetics" deviceset="GND" device=""/>
 <part name="GND44" library="SparkFun-Aesthetics" deviceset="GND" device=""/>
@@
 <part name="GND16" library="SparkFun-Aesthetics" deviceset="GND" device=""/>
 <part name="GND17" library="SparkFun-Aesthetics" deviceset="GND" device=""/>
-<part name="RS232_IND" library="MRDT-Connectors" deviceset="SL03" device=""/>
 <part name="RS232_PB" library="MRDT-Connectors" deviceset="SL03" device=""/>
 <part name="GND18" library="SparkFun-Aesthetics" deviceset="GND" device=""/>
 <part name="+3V7" library="supply1" deviceset="+3V3" device=""/>
+<part name="J1" library="MRDT-Connectors" deviceset="SL04" device="VERT"/>
+<part name="SUPPLY14" library="SparkFun-Aesthetics" deviceset="5V" device=""/>
 </parts>
 <sheets>
@@
 <instance part="U$14" gate="G$1" x="220.98" y="-342.9" rot="R90"/>
 <instance part="U$16" gate="G$1" x="416.56" y="-269.24" rot="MR180"/>
-<instance part="GND36" gate="1" x="594.36" y="-124.46"/>
+<instance part="GND36" gate="1" x="586.74" y="-134.62"/>
 <instance part="U2" gate="G$1" x="528.32" y="-99.06"/>
 <instance part="C44" gate="G$1" x="500.38" y="-83.82"/>
@@
 <instance part="GND16" gate="1" x="553.72" y="-83.82"/>
 <instance part="GND17" gate="1" x="553.72" y="-91.44"/>
-<instance part="RS232_IND" gate="G$1" x="607.06" y="-116.84"/>
 <instance part="RS232_PB" gate="G$1" x="607.06" y="-96.52"/>
 <instance part="GND18" gate="1" x="594.36" y="-104.14"/>
 <instance part="+3V7" gate="G$1" x="528.32" y="-55.88"/>
+<instance part="J1" gate="G$1" x="607.06" y="-124.46" rot="MR180"/>
+<instance part="SUPPLY14" gate="G$1" x="596.9" y="-116.84"/>
 </instances>
 <busses>
@@
 </segment>
 <segment>
-<pinref part="RS232_IND" gate="G$1" pin="1"/>
+<pinref part="J1" gate="G$1" pin="P$1"/>
 <pinref part="GND36" gate="1" pin="GND"/>
-<wire x1="599.44" y1="-119.38" x2="594.36" y2="-119.38" width="0.1524" layer="91"/>
-<wire x1="594.36" y1="-119.38" x2="594.36" y2="-121.92" width="0.1524" layer="91"/>
+<wire x1="599.44" y1="-132.08" x2="586.74" y2="-132.08" width="0.1524" layer="91"/>
 </segment>
 </net>
@@
 <net name="PACK_GATE" class="0">
 <segment>
-<label x="81.28" y="-99.06" size="1.778" layer="95"/>
 <pinref part="U$8" gate="G$1" pin="IN"/>
-<wire x1="81.28" y1="-99.06" x2="76.2" y2="-99.06" width="0.1524" layer="91"/>
+<wire x1="68.58" y1="-99.06" x2="76.2" y2="-99.06" width="0.1524" layer="91"/>
+<label x="68.58" y="-99.06" size="1.27" layer="95" rot="R180" xref="yes"/>
 </segment>
 <segment>
@@
 <wire x1="124.46" y1="-17.78" x2="111.76" y2="-17.78" width="0.1524" layer="91"/>
 </segment>
+<segment>
+<pinref part="J1" gate="G$1" pin="P$4"/>
+<pinref part="SUPPLY14" gate="G$1" pin="5V"/>
+<wire x1="599.44" y1="-116.84" x2="596.9" y2="-116.84" width="0.1524" layer="91"/>
+</segment>
 </net>
 <net name="LOGIC_POWER" class="0">
@@
 </segment>
 </net>
-<net name="BUZZ_1" class="0">
-<segment>
-<pinref part="Q11" gate="G$1" pin="G"/>
-<wire x1="414.02" y1="-200.66" x2="408.94" y2="-200.66" width="0.1524" layer="91"/>
-<label x="403.86" y="-200.66" size="1.778" layer="95" font="vector"/>
-<pinref part="R22" gate="G$1" pin="2"/>
-<wire x1="408.94" y1="-200.66" x2="403.86" y2="-200.66" width="0.1524" layer="91"/>
-<wire x1="408.94" y1="-203.2" x2="408.94" y2="-200.66" width="0.1524" layer="91"/>
-<junction x="408.94" y="-200.66"/>
-</segment>
-<segment>
-<pinref part="U$13" gate="G$1" pin="P4.7"/>
-<wire x1="419.1" y1="-78.74" x2="421.64" y2="-78.74" width="0.1524" layer="91"/>
-<label x="419.1" y="-78.74" size="1.27" layer="95" rot="R180" xref="yes"/>
-</segment>
-</net>
 <net name="GAUGE_ON" class="0">
 <segment>
@@
 </segment>
 <segment>
-<pinref part="RS232_IND" gate="G$1" pin="3"/>
-<wire x1="599.44" y1="-114.3" x2="591.82" y2="-114.3" width="0.1524" layer="91"/>
-<label x="591.82" y="-114.3" size="1.27" layer="95" rot="R180" xref="yes"/>
+<label x="584.2" y="-121.92" size="1.27" layer="95" rot="R180" xref="yes"/>
+<pinref part="J1" gate="G$1" pin="P$3"/>
+<wire x1="599.44" y1="-121.92" x2="584.2" y2="-121.92" width="0.1524" layer="91"/>
 </segment>
 </net>
@@
 </segment>
 <segment>
-<label x="591.82" y="-116.84" size="1.27" layer="95" rot="R180" xref="yes"/>
-<pinref part="RS232_IND" gate="G$1" pin="2"/>
-<wire x1="599.44" y1="-116.84" x2="591.82" y2="-116.84" width="0.1524" layer="91"/>
-</segment>
-</net>
+<label x="584.2" y="-127" size="1.27" layer="95" rot="R180" xref="yes"/>
+<pinref part="J1" gate="G$1" pin="P$2"/>
+<wire x1="599.44" y1="-127" x2="584.2" y2="-127" width="0.1524" layer="91"/>
+</segment>
+</net>
+<net name="BUZZER" class="0">
+<segment>
+<pinref part="U$13" gate="G$1" pin="P4.7"/>
+<wire x1="419.1" y1="-78.74" x2="421.64" y2="-78.74" width="0.1524" layer="91"/>
+<label x="419.1" y="-78.74" size="1.27" layer="95" rot="R180" xref="yes"/>
+</segment>
+<segment>
+<pinref part="Q11" gate="G$1" pin="G"/>
+<wire x1="414.02" y1="-200.66" x2="408.94" y2="-200.66" width="0.1524" layer="91"/>
+<label x="403.86" y="-200.66" size="1.778" layer="95" font="vector"/>
+<pinref part="R22" gate="G$1" pin="2"/>
+<wire x1="408.94" y1="-200.66" x2="403.86" y2="-200.66" width="0.1524" layer="91"/>
+<wire x1="408.94" y1="-203.2" x2="408.94" y2="-200.66" width="0.1524" layer="91"/>
+<junction x="408.94" y="-200.66"/>
+</segment>
+</net>

Commit message: Cleaned up routing
Parts:
- removed X5: 22-23-2041, con-molex:22-23-2041
- added D8: (no value), SparkFun-DiscreteSemi:DIODE1N4148
- added LOG_PWR: SL04VERT, MRDT-Connectors:SL04VERT
- C14: device rcl:C-USC1206 -> rcl:C-USC0805
- ESTOP_1, ESTOP_2: value M02POLAR -> SL02; device SparkFun-Connectors:M02POLAR -> MRDT-Connectors:SL02
- R25, R26, R27, R28, R38, R39: device resistor:R-US_R1206 -> rcl:R-US_R0805
- R40: device rcl:R-US_R1206 -> rcl:R-US_R0805
- renumbered J1 to RS232-IND, LED1 to V_OUT_LED, LED3 to LOG_PWR_LED
Connections:
- net 5V: now also D8.C, LOG_PWR.P$2; no longer X5-2.S
- net N$1: now also ESTOP_1.1; no longer ESTOP_2.2
- net N$2: now also LOG_PWR.P$4; no longer X5-4.S
- net N$34: now also ESTOP_2.2; no longer ESTOP_1.1
- net N$41: now also LOG_PWR.P$3; no longer X5-3.S
- net N$5: now also D8.A, LOG_PWR.P$1; no longer X5-1.S
Other:
- note added: "Coil"
- note removed: "Reset Coil"
- moved on the sheet: ESTOP_1, ESTOP_2, Q1, R23, R33
