File: Hardware/Main-BMS/BMS.brd (EAGLE design)
At the start: 114.3 x 124.5 mm, 97 parts, among them IC2 SMI-1324-TW-5V-2-R, J1 SL03, Q1 2N7002PW, Q10 2N7002PW, Q5 2N7002PW, Q6 2N7002PW, Q7 2N7002PW, Q8 2N7002PW, Q9 2N7002PW, U1 LT1910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

Commit message: Moved SLs on left edge of board farther right, checked for rev1 board ordering with Jacob.
Parts:
- moved U$1 17.6 mm to (44.5, 14.0), turned to 0 degrees
- moved J1 7.62 mm to (20.3, 55.6)
- moved RS232_PB 7.62 mm to (20.4, 33.0)
- moved D10 5.06 mm to (12.4, 55.6), turned to 180 degrees
- moved D11 4.50 mm to (21.6, 60.2), turned to 0 degrees
Routing:
- net RS232_RX_PB: track 21.2 -> 12.5 mm
- net RS232_TX_PB: track 15.9 -> 21.8 mm
- net SER_TX_IND: track 94.1 -> 90.3 mm
- net +3V3: track 111.3 -> 107.7 mm
- net N$3: vias 22 -> 24
- net GND: vias 86 -> 84
