File: _saved_BMS_Hardware.sch (KiCad schematic (older format))
At the start: 4 parts

Commit message: Started Schematic and Layout
Parts:
- gave numbers to parts that had none: 1
Changed lines of the file:
@@
 $EndComp
 $Comp
-L LT1910 U?
+L LT1910 U1
 U 1 1 5ACD5F48
 P 4950 2200
-F 0 "U?" H 5000 2150 60  0000 C CNN
+F 0 "U1" H 5000 2150 60  0000 C CNN
 F 1 "LT1910" H 5100 2750 60  0000 C CNN
 F 2 "" H 4950 2200 60  0001 C CNN
