File: BMS_Hardware.sch (KiCad schematic (older format))
At the start: 123 parts, among them Q1 2N7002PW, Q2 2N7002PW, Q3 2N7002PW, Q4 2N7002PW, Q5 2N7002PW, Q6 IRLS3034-7P, Q7 IRLS3034-7P, Q8 2N7002PW, Q9 2N7002PW, U1 ACS759ECB-200B-PFF-T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

Commit message: finished the cells
Parts:
- removed C2, C3, C4, C5, C6, C7, C8: 100n, Capacitors_SMD:C_0603_HandSoldering, symbol BMS_Hardware-rescue:C
- removed D2, D3, D4, D5, D6, D7, D8: 7.5V, Diodes_SMD:D_SOD-323_HandSoldering, symbol BMS_Hardware-rescue:D_Zener
- removed R2, R3, R4, R5, R6, R7, R8: 100, Resistors_SMD:R_0603_HandSoldering, symbol BMS_Hardware-rescue:R
- added R? (x8): 21.5k, symbol BMS_Hardware-rescue:R
- added R? (x8): 78.7k, symbol BMS_Hardware-rescue:R
Connections:
- net labels removed: CELL_1_FILTER, CELL_2_FILTER, CELL_3_FILTER, CELL_4_FILTER, CELL_5_FILTER, CELL_6_FILTER, CELL_7_FILTER, CELL_8_FILTER
- wire segments 334 -> 315
Other:
- moved on the sheet: C?, D?

Commit message: Added Diodes to voltage dividers
Parts:
- added D? (x10): D_Schottky, symbol Device:D_Schottky
- C1: value 100n -> 1u
Connections:
- wire segments 315 -> 316
Other:
- moved on the sheet: R22, R23
Changed lines of the file:
@@
 	6850 2650 7300 2650
-Wire Wire Line
-	8800 2650 9500 2650
 Wire Wire Line
 	7200 2150 7300 2150
@@
 L BMS_Hardware-rescue:R R22
 U 1 1 5AD5C40D
-P 9500 2950
-F 0 "R22" V 9400 2950 50  0000 C CNN
-F 1 "1M" V 9500 2950 50  0000 C CNN
-F 2 "Resistors_SMD:R_0603_HandSoldering" V 9430 2950 50  0001 C CNN
-F 3 "" H 9500 2950 50  0001 C CNN
-	1    9500 2950
+P 9600 2950
+F 0 "R22" V 9500 2950 50  0000 C CNN
+F 1 "1M" V 9600 2950 50  0000 C CNN
+F 2 "Resistors_SMD:R_0603_HandSoldering" V 9530 2950 50  0001 C CNN
+F 3 "" H 9600 2950 50  0001 C CNN
+	1    9600 2950
 	1    0    0    -1
 $EndComp
@@
 L BMS_Hardware-rescue:R R23
 U 1 1 5AD5C4DB
-P 9500 3450
-F 0 "R23" V 9400 3450 50  0000 C CNN
-F 1 "100k" V 9500 3450 50  0000 C CNN
-F 2 "Resistors_SMD:R_0603_HandSoldering" V 9430 3450 50  0001 C CNN
-F 3 "" H 9500 3450 50  0001 C CNN
-	1    9500 3450
-	1    0    0    -1
-$EndComp
-Wire Wire Line
-	9500 3100 9500 3200
-Wire Wire Line
-	9500 3600 9500 3700
-Text GLabel 9500 3700 0    60   UnSpc ~ 0
-GND
-Wire Wire Line
-	9500 2650 9500 2800
-Wire Wire Line
-	9500 3200 9600 3200
-Connection ~ 9500 3200
-Text GLabel 9600 3200 2    60   Output ~ 0
+P 9750 3450
+F 0 "R23" V 9650 3450 50  0000 C CNN
+F 1 "100k" V 9750 3450 50  0000 C CNN
+F 2 "Resistors_SMD:R_0603_HandSoldering" V 9680 3450 50  0001 C CNN
+F 3 "" H 9750 3450 50  0001 C CNN
+	1    9750 3450
+	0    1    1    0
+$EndComp
+Wire Wire Line
+	9600 3100 9600 3200
+Text GLabel 9900 3450 2    60   UnSpc ~ 0
+GND
+Wire Wire Line
+	9600 2650 9600 2800
+Wire Wire Line
+	9600 3200 9700 3200
+Connection ~ 9600 3200
+Text GLabel 9700 3200 2    60   Output ~ 0
 V_CHECK_OUT
 $Comp
@@
 Text GLabel 4850 1750 2    60   Output ~ 0
 V_CHECK_ARRAY
-Connection ~ 9500 2650
 Text GLabel 9800 2650 2    60   Output ~ 0
 V_OUT
@@
 P 2400 5550
 F 0 "C1" H 2410 5620 50  0000 L CNN
-F 1 "100n" H 2410 5470 50  0000 L CNN
+F 1 "1u" H 2410 5470 50  0000 L CNN
 F 2 "Capacitors_SMD:C_0603_HandSoldering" H 2400 5550 50  0001 C CNN
 F 3 "" H 2400 5550 50  0001 C CNN
@@
 	7000 2950 7000 4450
 Wire Wire Line
-	9500 3200 9500 3300
-Wire Wire Line
 	4050 2650 6350 2650
 Wire Wire Line
@@
 Wire Wire Line
 	4800 1750 4800 1800
-Wire Wire Line
-	9500 2650 9700 2650
 Wire Wire Line
 	14250 1900 14500 1900
@@
 Text GLabel 3300 10600 0    50   UnSpc ~ 0
 GND
-Text GLabel 4750 10300 2    50   Output ~ 0
+Text GLabel 5300 10500 2    50   Output ~ 0
 CELL_8-7
 Wire Wire Line
@@
 Text GLabel 3300 6300 0    50   UnSpc ~ 0
 GND
-Text GLabel 4750 9550 2    50   Output ~ 0
+Text GLabel 5300 9750 2    50   Output ~ 0
 CELL_7-6
-Text GLabel 4750 8800 2    50   Output ~ 0
+Text GLabel 5300 9000 2    50   Output ~ 0
 CELL_6-5
-Text GLabel 4750 8100 2    50   Output ~ 0
+Text GLabel 5300 8300 2    50   Output ~ 0
 CELL_5-4
-Text GLabel 4750 7400 2    50   Output ~ 0
+Text GLabel 5300 7600 2    50   Output ~ 0
 CELL_4-3
-Text GLabel 4750 6700 2    50   Output ~ 0
+Text GLabel 5300 6900 2    50   Output ~ 0
 CELL_3-2
-Text GLabel 4750 6000 2    50   Output ~ 0
+Text GLabel 5350 6200 2    50   Output ~ 0
 CELL_2-1
 Wire Wire Line
@@
 	2050 9400 2800 9400
 Connection ~ 2400 5350
-Text GLabel 3150 5200 2    50   Output ~ 0
+Text GLabel 3700 5400 2    50   Output ~ 0
 CELL_1-GND
 Text GLabel 2050 5700 0    50   Input ~ 0
@@
 $EndComp
 Wire Wire Line
-	3150 5400 3150 5200
-Wire Wire Line
 	3150 5400 3450 5400
-Connection ~ 3150 5400
 Text GLabel 3450 5700 2    50   UnSpc ~ 0
 GND
@@
 $EndComp
 Wire Wire Line
-	4750 6200 4750 6000
-Wire Wire Line
 	4750 6200 5050 6200
-Connection ~ 4750 6200
 Text GLabel 5050 6500 2    50   UnSpc ~ 0
 GND
@@
 $EndComp
 Wire Wire Line
-	4750 6900 4750 6700
-Wire Wire Line
 	4750 6900 5050 6900
-Connection ~ 4750 6900
 Text GLabel 5050 7200 2    50   UnSpc ~ 0
 GND
@@
 $EndComp
 Wire Wire Line
-	4750 7600 4750 7400
-Wire Wire Line
 	4750 7600 5050 7600
-Connection ~ 4750 7600
 Text GLabel 5050 7900 2    50   UnSpc ~ 0
 GND
@@
 $EndComp
 Wire Wire Line
-	4750 8300 4750 8100
-Wire Wire Line
 	4750 8300 5050 8300
-Connection ~ 4750 8300
 Text GLabel 5050 8600 2    50   UnSpc ~ 0
 GND
@@
 $EndComp
 Wire Wire Line
-	4750 9000 4750 8800
-Wire Wire Line
 	4750 9000 5050 9000
-Connection ~ 4750 9000
 Text GLabel 5050 9300 2    50   UnSpc ~ 0
 GND
@@
 $EndComp
 Wire Wire Line
-	4750 9750 4750 9550
-Wire Wire Line
 	4750 9750 5050 9750
-Connection ~ 4750 9750
 Text GLabel 5050 10050 2    50   UnSpc ~ 0
 GND
@@
 $EndComp
 Wire Wire Line
-	4750 10500 4750 10300
-Wire Wire Line
 	4750 10500 5050 10500
-Connection ~ 4750 10500
 Text GLabel 5050 10800 2    50   UnSpc ~ 0
 GND
@@
 Wire Wire Line
 	2800 10150 3000 10150
+Text GLabel 3150 5100 0    50   Input ~ 0
+3V3
+$Comp
+L Device:D_Schottky D?
+U 1 1 5BCDE88D
+P 3150 5250
+F 0 "D?" V 3104 5329 50  0000 L CNN
+F 1 "D_Schottky" V 3195 5329 50  0000 L CNN
+F 2 "" H 3150 5250 50  0001 C CNN
+F 3 "~" H 3150 5250 50  0001 C CNN
+	1    3150 5250
+	0    1    1    0
+$EndComp
+Connection ~ 3150 5400
+Text GLabel 4750 5900 0    50   Input ~ 0
+3V3
+$Comp
+L Device:D_Schottky D?
+U 1 1 5BDC82AB
+P 4750 6050
+F 0 "D?" V 4704 6129 50  0000 L CNN
+F 1 "D_Schottky" V 4795 6129 50  0000 L CNN
+F 2 "" H 4750 6050 50  0001 C CNN
+F 3 "~" H 4750 6050 50  0001 C CNN
+	1    4750 6050
+	0    1    1    0
+$EndComp
+$Comp
+L Device:D_Schottky D?
+U 1 1 5BE0A38D
+P 4750 6750
+F 0 "D?" V 4704 6829 50  0000 L CNN
+F 1 "D_Schottky" V 4795 6829 50  0000 L CNN
+F 2 "" H 4750 6750 50  0001 C CNN
+F 3 "~" H 4750 6750 50  0001 C CNN
+	1    4750 6750
+	0    1    1    0
+$EndComp
+$Comp
+L Device:D_Schottky D?
+U 1 1 5BE0A481
+P 4750 7450
+F 0 "D?" V 4704 7529 50  0000 L CNN
+F 1 "D_Schottky" V 4795 7529 50  0000 L CNN
+F 2 "" H 4750 7450 50  0001 C CNN
+F 3 "~" H 4750 7450 50  0001 C CNN
+	1    4750 7450
+	0    1    1    0
+$EndComp
+$Comp
+L Device:D_Schottky D?
+U 1 1 5BE0A65B
+P 4750 8150
+F 0 "D?" V 4704 8229 50  0000 L CNN
+F 1 "D_Schottky" V 4795 8229 50  0000 L CNN
+F 2 "" H 4750 8150 50  0001 C CNN
+F 3 "~" H 4750 8150 50  0001 C CNN
+	1    4750 8150
+	0    1    1    0
+$EndComp
+$Comp
+L Device:D_Schottky D?
+U 1 1 5BE0A751
+P 4750 8850
+F 0 "D?" V 4704 8929 50  0000 L CNN
+F 1 "D_Schottky" V 4795 8929 50  0000 L CNN
+F 2 "" H 4750 8850 50  0001 C CNN
+F 3 "~" H 4750 8850 50  0001 C CNN
+	1    4750 8850
+	0    1    1    0
+$EndComp
+$Comp
+L Device:D_Schottky D?
+U 1 1 5BE0B244
+P 4750 9600
+F 0 "D?" V 4704 9679 50  0000 L CNN
+F 1 "D_Schottky" V 4795 9679 50  0000 L CNN
+F 2 "" H 4750 9600 50  0001 C CNN
+F 3 "~" H 4750 9600 50  0001 C CNN
+	1    4750 9600
+	0    1    1    0
+$EndComp
+$Comp
+L Device:D_Schottky D?
+U 1 1 5BE0B346
+P 4750 10350
+F 0 "D?" V 4704 10429 50  0000 L CNN
+F 1 "D_Schottky" V 4795 10429 50  0000 L CNN
+F 2 "" H 4750 10350 50  0001 C CNN
+F 3 "~" H 4750 10350 50  0001 C CNN
+	1    4750 10350
+	0    1    1    0
+$EndComp
+Text GLabel 4750 6600 0    50   Input ~ 0
+3V3
+Text GLabel 4750 7300 0    50   Input ~ 0
+3V3
+Text GLabel 4750 8000 0    50   Input ~ 0
+3V3
+Text GLabel 4750 8700 0    50   Input ~ 0
+3V3
+Text GLabel 4750 9450 0    50   Input ~ 0
+3V3
+Text GLabel 4750 10200 0    50   Input ~ 0
+3V3
+Connection ~ 4750 6200
+Wire Wire Line
+	5050 6200 5350 6200
+Connection ~ 5050 6200
+Wire Wire Line
+	3450 5400 3700 5400
+Connection ~ 3450 5400
+Connection ~ 4750 6900
+Wire Wire Line
+	5050 6900 5300 6900
+Connection ~ 5050 6900
+Connection ~ 4750 7600
+Wire Wire Line
+	5050 7600 5300 7600
+Connection ~ 5050 7600
+Connection ~ 4750 8300
+Wire Wire Line
+	5050 8300 5300 8300
+Connection ~ 5050 8300
+Connection ~ 4750 9000
+Wire Wire Line
+	5300 9000 5050 9000
+Connection ~ 5050 9000
+Connection ~ 4750 9750
+Wire Wire Line
+	5050 9750 5300 9750
+Connection ~ 5050 9750
+Connection ~ 4750 10500
+Wire Wire Line
+	5050 10500 5300 10500
+Connection ~ 5050 10500
+Connection ~ 9600 2650
+Wire Wire Line
+	9600 2650 9700 2650
+Wire Wire Line
+	8800 2650 9600 2650
+Wire Wire Line
+	9600 3200 9300 3200
+Wire Wire Line
+	9300 3200 9300 3400
+$Comp
+L Device:D_Schottky D?
+U 1 1 5C0B6592
+P 9300 3550
+F 0 "D?" V 9346 3471 50  0000 R CNN
+F 1 "D_Schottky" V 9255 3471 50  0000 R CNN
+F 2 "" H 9300 3550 50  0001 C CNN
+F 3 "~" H 9300 3550 50  0001 C CNN
+	1    9300 3550
+	0    -1   -1   0
+$EndComp
+Wire Wire Line
+	9600 3200 9600 3450
+$Comp
+L Device:D_Schottky D?
+U 1 1 5C11FFF1
+P 4200 1750
+F 0 "D?" V 4246 1671 50  0000 R CNN
+F 1 "D_Schottky" V 4155 1671 50  0000 R CNN
+F 2 "" H 4200 1750 50  0001 C CNN
+F 3 "~" H 4200 1750 50  0001 C CNN
+	1    4200 1750
+	0    -1   -1   0
+$EndComp
 $EndSCHEMATC

Commit message: finished all voltage dividers
Parts:
- added D? (x2): D_Schottky, symbol Device:D_Schottky
Connections:
- wire segments 316 -> 319
Other:
- moved on the sheet: R18
Changed lines of the file:
@@
 L BMS_Hardware-rescue:R R18
 U 1 1 5AD54C65
-P 5600 3800
-F 0 "R18" V 5500 3800 50  0000 C CNN
-F 1 "4k" V 5600 3800 50  0000 C CNN
-F 2 "Resistors_SMD:R_0603_HandSoldering" V 5530 3800 50  0001 C CNN
-F 3 "" H 5600 3800 50  0001 C CNN
-	1    5600 3800
+P 5400 3800
+F 0 "R18" V 5300 3800 50  0000 C CNN
+F 1 "4k" V 5400 3800 50  0000 C CNN
+F 2 "Resistors_SMD:R_0603_HandSoldering" V 5330 3800 50  0001 C CNN
+F 3 "" H 5400 3800 50  0001 C CNN
+	1    5400 3800
 	0    1    1    0
 $EndComp
-Wire Wire Line
-	5850 3800 5750 3800
 Connection ~ 5850 3800
 Wire Wire Line
@@
 Connection ~ 5850 4150
 Wire Wire Line
-	5450 3800 5400 3800
-Text GLabel 5400 3800 0    60   Input ~ 0
+	5250 3800 5200 3800
+Text GLabel 5200 3800 0    60   Input ~ 0
 V_OUT
 $Comp
@@
 	0    -1   -1   0
 $EndComp
-Wire Wire Line
-	4050 1200 4050 2650
 Connection ~ 4050 2650
 Wire Wire Line
@@
 Wire Wire Line
 	9600 3200 9300 3200
-Wire Wire Line
-	9300 3200 9300 3400
 $Comp
 L Device:D_Schottky D?
 U 1 1 5C0B6592
-P 9300 3550
-F 0 "D?" V 9346 3471 50  0000 R CNN
-F 1 "D_Schottky" V 9255 3471 50  0000 R CNN
-F 2 "" H 9300 3550 50  0001 C CNN
-F 3 "~" H 9300 3550 50  0001 C CNN
-	1    9300 3550
+P 9300 3350
+F 0 "D?" V 9346 3271 50  0000 R CNN
+F 1 "D_Schottky" H 9255 3271 50  0000 R CNN
+F 2 "" H 9300 3350 50  0001 C CNN
+F 3 "~" H 9300 3350 50  0001 C CNN
+	1    9300 3350
 	0    -1   -1   0
 $EndComp
@@
 L Device:D_Schottky D?
 U 1 1 5C11FFF1
-P 4200 1750
-F 0 "D?" V 4246 1671 50  0000 R CNN
-F 1 "D_Schottky" V 4155 1671 50  0000 R CNN
-F 2 "" H 4200 1750 50  0001 C CNN
-F 3 "~" H 4200 1750 50  0001 C CNN
-	1    4200 1750
+P 4650 1750
+F 0 "D?" V 4696 1671 50  0000 R CNN
+F 1 "D_Schottky" H 4605 1671 50  0000 R CNN
+F 2 "" H 4650 1750 50  0001 C CNN
+F 3 "~" H 4650 1750 50  0001 C CNN
+	1    4650 1750
+	1    0    0    -1
+$EndComp
+Text GLabel 9300 3500 3    49   Input ~ 0
+3V3
+Text GLabel 4500 1750 0    49   Input ~ 0
+3V3
+Wire Wire Line
+	4050 1200 4050 2650
+Wire Wire Line
+	15150 3900 15450 3900
+$Comp
+L Device:D_Schottky D?
+U 1 1 5C286B97
+P 15450 4050
+F 0 "D?" V 15496 3971 50  0000 R CNN
+F 1 "D_Schottky" H 15405 3971 50  0000 R CNN
+F 2 "" H 15450 4050 50  0001 C CNN
+F 3 "~" H 15450 4050 50  0001 C CNN
+	1    15450 4050
 	0    -1   -1   0
 $EndComp
+Text GLabel 15450 4200 3    49   Input ~ 0
+3V3
+Wire Wire Line
+	5550 3800 5650 3800
+Wire Wire Line
+	5650 4000 5600 4000
+Wire Wire Line
+	5650 3800 5650 4000
+Connection ~ 5650 3800
+Wire Wire Line
+	5650 3800 5850 3800
+$Comp
+L Device:D_Schottky D?
+U 1 1 5C39F088
+P 5450 4000
+F 0 "D?" V 5496 3921 50  0000 R CNN
+F 1 "D_Schottky" H 5405 3921 50  0000 R CNN
+F 2 "" H 5450 4000 50  0001 C CNN
+F 3 "~" H 5450 4000 50  0001 C CNN
+	1    5450 4000
+	1    0    0    -1
+$EndComp
+Text GLabel 5300 4000 0    49   Input ~ 0
+3V3
 $EndSCHEMATC

Commit message: Created .txt file for pin layout
Parts:
- R1, R16, R3, R4, R5, R6, R7, R8: renamed from R?; value 21.5k -> 10k
- R17, R2, R21, R30, R31, R32, R33, R34: renamed from R?; value 78.7k -> 36.5k
- gave numbers to parts that had none: 34
Connections:
- net labels removed: ADC_CELL_A0, ADC_CELL_A1, ADC_CELL_A2, ADC_CELL_EN, ADC_CELL_VOUT, SER_RX_PB, SER_TX_PB, TM4C1294NCPDT
- wire segments 319 -> 377
- no-connect marks 0 -> 63
Other:
- note added: "TM4C1294NCPDT"

Commit message: footprints
Parts:
- C1, C10, C18, C19, C20, C23, C27, C28, C29, C30, C31: footprint Capacitors_SMD:C_0603_HandSoldering -> Capacitor_SMD:C_0603_1608Metric_Pad1.05x0.95mm_HandSolder
- C11, C12, C13, C14, C15, C16, C2, C3, C4, C5, C6, C7, C8, C9: footprint (none) -> Capacitor_SMD:C_0603_1608Metric_Pad1.05x0.95mm_HandSolder
- C17, C26: footprint Capacitors_THT:CP_Radial_D6.3mm_P2.50mm -> Capacitor_THT:CP_Radial_D6.3mm_P2.50mm
- Conn1, Conn2: footprint MRDT_Connectors:MOLEX_SL_9_Vertical -> MRDT_Connectors:MOLEX_SL_09_Vertical
- D1, D11, D2, D3, D4, D5, D6, D7, D8: footprint Diodes_SMD:D_SOD-323_HandSoldering -> Diode_SMD:D_SOD-323_HandSoldering
- D12, D13, D14, D15, D16, D17, D18, D19, D20, D21, D22, D23: footprint (none) -> Diode_SMD:D_0603_1608Metric_Pad1.05x0.95mm_HandSolder
- R1, R16, R17, R2, R21, R29, R3, R30, R31, R32, R33, R34, R4, R5, R6, R7, R8: footprint (none) -> Resistor_SMD:R_0603_1608Metric_Pad1.05x0.95mm_HandSolder
- R10, R11, R12, R13, R14, R15, R18, R19, R20, R22, R23, R24, R25, R26, R27, R28, R9: footprint Resistors_SMD:R_0603_HandSoldering -> Resistor_SMD:R_0603_1608Metric_Pad1.05x0.95mm_HandSolder
- U10, U5: footprint MRDT_Connectors:MOLEX_SL_4_Vertical -> MRDT_Connectors:MOLEX_SL_04_Vertical
- U11: footprint MRDT_Connectors:MOLEX_SL_3_Vertical -> MRDT_Connectors:MOLEX_SL_03_Vertical
- U12, U2, U4, U7, U8: footprint MRDT_Connectors:MOLEX_SL_2_Vertical -> MRDT_Connectors:MOLEX_SL_02_Vertical
- U13, U14, U15, U19, U20, U3, U9: footprint (none) -> Package_SO:SO-8_5.3x6.2mm_P1.27mm
- U21: footprint (none) -> MRDT_Shields:TM4C129E_Launchpad_FULL_Bottom_SMD

Commit message: footprints
Parts:
- C24: footprint Capacitors_SMD:C_0603_HandSoldering -> Capacitor_SMD:C_0603_1608Metric_Pad1.05x0.95mm_HandSolder
- D10, D9: footprint LEDs:LED_0603_HandSoldering -> LED_SMD:LED_0603_1608Metric_Pad1.05x0.95mm_HandSolder
- F1: footprint Fuse_Holders_and_Fuses:Fuse_SMD2920 -> Fuse:Fuse_2920_7451Metric
- U17: footprint MRDT_Connectors:MOLEX_SL_3_Vertical -> MRDT_Connectors:MOLEX_SL_03_Vertical
- U18: footprint MRDT_Devices:OKI_Horisontal -> MRDT_Devices:OKI_Horizontal
Changed lines of the file:
@@
 F 0 "U18" H 13950 1050 60  0001 C CNN
 F 1 "OKI" H 14250 1650 60  0000 C CNN
-F 2 "MRDT_Devices:OKI_Horisontal" H 13850 1200 60  0001 C CNN
+F 2 "MRDT_Devices:OKI_Horizontal" H 13850 1200 60  0001 C CNN
 F 3 "" H 13850 1200 60  0001 C CNN
 	1    14100 1300
@@
 F 0 "F1" V 4350 1250 50  0000 C CNN
 F 1 "PTC2920" V 4550 1250 50  0000 C CNN
-F 2 "Fuse_Holders_and_Fuses:Fuse_SMD2920" H 4500 1050 50  0001 L CNN
+F 2 "Fuse:Fuse_2920_7451Metric" H 4500 1050 50  0001 L CNN
 F 3 "" H 4450 1250 50  0001 C CNN
 	1    4450 1250
@@
 F 0 "C24" H 12810 1820 50  0000 L CNN
 F 1 "0.1u" H 12810 1670 50  0000 L CNN
-F 2 "Capacitors_SMD:C_0603_HandSoldering" H 12800 1750 50  0001 C CNN
+F 2 "Capacitor_SMD:C_0603_1608Metric_Pad1.05x0.95mm_HandSolder" H 12800 1750 50  0001 C CNN
 F 3 "" H 12800 1750 50  0001 C CNN
 	1    12800 1750
@@
 F 0 "U17" H 11350 3650 60  0001 C CNN
 F 1 "Indicator Comm" H 11350 4050 60  0000 C CNN
-F 2 "MRDT_Connectors:MOLEX_SL_3_Vertical" H 11300 3700 60  0001 C CNN
+F 2 "MRDT_Connectors:MOLEX_SL_03_Vertical" H 11300 3700 60  0001 C CNN
 F 3 "" H 11300 3700 60  0001 C CNN
 	1    11300 3700
@@
 F 0 "D9" H 13500 3300 50  0000 C CNN
 F 1 "LOG_PWR_LED" H 13500 3100 50  0000 C CNN
-F 2 "LEDs:LED_0603_HandSoldering" H 13500 3200 50  0001 C CNN
+F 2 "LED_SMD:LED_0603_1608Metric_Pad1.05x0.95mm_HandSolder" H 13500 3200 50  0001 C CNN
 F 3 "" H 13500 3200 50  0001 C CNN
 	1    13500 3200
@@
 F 0 "D10" H 14450 3150 50  0000 C CNN
 F 1 "V_OUT_LED" H 14450 2950 50  0000 C CNN
-F 2 "LEDs:LED_0603_HandSoldering" H 14450 3050 50  0001 C CNN
+F 2 "LED_SMD:LED_0603_1608Metric_Pad1.05x0.95mm_HandSolder" H 14450 3050 50  0001 C CNN
 F 3 "" H 14450 3050 50  0001 C CNN
 	1    14450 3050
