File: BMS_Hardware.sch (KiCad schematic (older format))
At the start: 123 parts, among them Q1 2N7002PW, Q2 2N7002PW, Q3 2N7002PW, Q4 2N7002PW, Q5 2N7002PW, Q6 IRLS3034-7P, Q7 IRLS3034-7P, Q8 2N7002PW, Q9 2N7002PW, U1 ACS759ECB-200B-PFF-T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

Commit message: Added Tiva_Top_SMD; Loaded board layout
Libraries are not mapped correctly, the layout cannot pull correct packages
Parts:
- U21: footprint MRDT_Shields:TM4C129E_Launchpad_FULL_Bottom_SMD -> BMS_Hardware:TM4C129E_Launchpad_FULL_Top_SMD
Other:
- moved on the sheet: C1, D1, R1, R2
Changed lines of the file:
@@
 L BMS_Hardware-rescue:D_Zener D1
 U 1 1 5ACFDF7D
-P 2750 5550
-F 0 "D1" H 2750 5650 50  0000 C CNN
-F 1 "7.5V" H 2750 5450 50  0000 C CNN
-F 2 "Diode_SMD:D_SOD-323_HandSoldering" H 2750 5550 50  0001 C CNN
-F 3 "" H 2750 5550 50  0001 C CNN
-	1    2750 5550
+P 2650 5700
+F 0 "D1" H 2650 5800 50  0000 C CNN
+F 1 "7.5V" H 2650 5600 50  0000 C CNN
+F 2 "Diode_SMD:D_SOD-323_HandSoldering" H 2650 5700 50  0001 C CNN
+F 3 "" H 2650 5700 50  0001 C CNN
+	1    2650 5700
 	0    -1   -1   0
 $EndComp
-Connection ~ 2400 5700
-Wire Wire Line
-	2400 5400 2400 5350
-Text GLabel 2400 5250 2    60   UnSpc ~ 0
-GND
-Wire Wire Line
-	2750 5400 2750 5350
-Wire Wire Line
-	2750 5350 2400 5350
+Connection ~ 2300 5850
+Wire Wire Line
+	2300 5550 2300 5500
+Text GLabel 2300 5400 2    60   UnSpc ~ 0
+GND
+Wire Wire Line
+	2650 5550 2650 5500
+Wire Wire Line
+	2650 5500 2300 5500
 Text GLabel 1950 6600 0    51   Input ~ 0
 CELL_2
@@
 L BMS_Hardware-rescue:C C1
 U 1 1 5ADAB430
-P 2400 5550
-F 0 "C1" H 2410 5620 50  0000 L CNN
-F 1 "1u" H 2410 5470 50  0000 L CNN
-F 2 "Capacitor_SMD:C_0603_1608Metric_Pad1.05x0.95mm_HandSolder" H 2400 5550 50  0001 C CNN
-F 3 "" H 2400 5550 50  0001 C CNN
-	1    2400 5550
+P 2300 5700
+F 0 "C1" H 2310 5770 50  0000 L CNN
+F 1 "1u" H 2310 5620 50  0000 L CNN
+F 2 "Capacitor_SMD:C_0603_1608Metric_Pad1.05x0.95mm_HandSolder" H 2300 5700 50  0001 C CNN
+F 3 "" H 2300 5700 50  0001 C CNN
+	1    2300 5700
 	-1   0    0    1
 $EndComp
@@
 	1050 3050 1050 3200
 Wire Wire Line
-	2400 5700 2050 5700
-Wire Wire Line
-	2750 5700 2400 5700
-Wire Wire Line
-	2400 5350 2400 5250
+	2300 5850 1950 5850
+Wire Wire Line
+	2650 5850 2300 5850
+Wire Wire Line
+	2300 5500 2300 5400
 Wire Wire Line
 	7950 9250 8050 9250
@@
 F 0 "U21" H 13550 8150 60  0000 L CNN
 F 1 "TM4C129E_Launchpad" H 13200 8050 60  0000 L CNN
-F 2 "MRDT_Shields:TM4C129E_Launchpad_FULL_Bottom_SMD" H 13900 6900 60  0001 C CNN
+F 2 "BMS_Hardware:TM4C129E_Launchpad_FULL_Top_SMD" H 13900 6900 60  0001 C CNN
 F 3 "" H 13900 6900 60  0001 C CNN
 	3    13900 6900
@@
 F 0 "U21" H 14200 8150 60  0000 C CNN
 F 1 "TM4C129E_Launchpad" H 14150 8050 60  0000 C CNN
-F 2 "MRDT_Shields:TM4C129E_Launchpad_FULL_Bottom_SMD" H 14500 6900 60  0001 C CNN
+F 2 "BMS_Hardware:TM4C129E_Launchpad_FULL_Top_SMD" H 14500 6900 60  0001 C CNN
 F 3 "" H 14500 6900 60  0001 C CNN
 	4    14500 6900
@@
 F 0 "U21" H 11050 10400 60  0000 L CNN
 F 1 "TM4C129E_Launchpad" H 10700 10300 60  0000 L CNN
-F 2 "MRDT_Shields:TM4C129E_Launchpad_FULL_Bottom_SMD" H 11450 9150 60  0001 C CNN
+F 2 "BMS_Hardware:TM4C129E_Launchpad_FULL_Top_SMD" H 11450 9150 60  0001 C CNN
 F 3 "" H 11450 9150 60  0001 C CNN
 	5    11450 9150
@@
 F 0 "U21" H 11850 10400 60  0000 C CNN
 F 1 "TM4C129E_Launchpad" H 11800 10300 60  0000 C CNN
-F 2 "MRDT_Shields:TM4C129E_Launchpad_FULL_Bottom_SMD" H 12050 9150 60  0001 C CNN
+F 2 "BMS_Hardware:TM4C129E_Launchpad_FULL_Top_SMD" H 12050 9150 60  0001 C CNN
 F 3 "" H 12050 9150 60  0001 C CNN
 	6    12050 9150
@@
 F 0 "U21" H 13850 10400 60  0000 L CNN
 F 1 "TM4C129E_Launchpad" H 13400 10300 60  0000 L CNN
-F 2 "MRDT_Shields:TM4C129E_Launchpad_FULL_Bottom_SMD" H 14100 9150 60  0001 C CNN
+F 2 "BMS_Hardware:TM4C129E_Launchpad_FULL_Top_SMD" H 14100 9150 60  0001 C CNN
 F 3 "" H 14100 9150 60  0001 C CNN
 	7    14100 9150
@@
 F 0 "U21" H 14550 10400 60  0000 C CNN
 F 1 "TM4C129E_Launchpad" H 14450 10300 60  0000 C CNN
-F 2 "MRDT_Shields:TM4C129E_Launchpad_FULL_Bottom_SMD" H 14700 9150 60  0001 C CNN
+F 2 "BMS_Hardware:TM4C129E_Launchpad_FULL_Top_SMD" H 14700 9150 60  0001 C CNN
 F 3 "" H 14700 9150 60  0001 C CNN
 	8    14700 9150
@@
 F 0 "U21" H 11200 8150 60  0000 L CNN
 F 1 "TM4C129E_Launchpad" H 10800 8050 60  0000 L CNN
-F 2 "MRDT_Shields:TM4C129E_Launchpad_FULL_Bottom_SMD" H 11550 6900 60  0001 C CNN
+F 2 "BMS_Hardware:TM4C129E_Launchpad_FULL_Top_SMD" H 11550 6900 60  0001 C CNN
 F 3 "" H 11550 6900 60  0001 C CNN
 	1    11550 6900
@@
 F 0 "U21" H 12050 8150 60  0000 C CNN
 F 1 "TM4C129E_Launchpad" H 11950 8050 60  0000 C CNN
-F 2 "MRDT_Shields:TM4C129E_Launchpad_FULL_Bottom_SMD" H 12150 6900 60  0001 C CNN
+F 2 "BMS_Hardware:TM4C129E_Launchpad_FULL_Top_SMD" H 12150 6900 60  0001 C CNN
 F 3 "" H 12150 6900 60  0001 C CNN
 	2    12150 6900
@@
 Wire Wire Line
 	2050 9400 2800 9400
-Connection ~ 2400 5350
-Text GLabel 3700 5400 2    50   Output ~ 0
+Connection ~ 2300 5500
+Text GLabel 3600 5550 2    50   Output ~ 0
 CELL_1-GND
-Text GLabel 2050 5700 0    50   Input ~ 0
+Text GLabel 1950 5850 0    50   Input ~ 0
 CELL_1
 $Comp
 L BMS_Hardware-rescue:R R1
 U 1 1 5BC6068A
-P 3150 5550
-F 0 "R1" H 3220 5596 50  0000 L CNN
-F 1 "10k" H 3220 5505 50  0000 L CNN
-F 2 "Resistor_SMD:R_0603_1608Metric_Pad1.05x0.95mm_HandSolder" V 3080 5550 50  0001 C CNN
-F 3 "" H 3150 5550 50  0001 C CNN
-	1    3150 5550
+P 3050 5700
+F 0 "R1" H 3120 5746 50  0000 L CNN
+F 1 "10k" H 3120 5655 50  0000 L CNN
+F 2 "Resistor_SMD:R_0603_1608Metric_Pad1.05x0.95mm_HandSolder" V 2980 5700 50  0001 C CNN
+F 3 "" H 3050 5700 50  0001 C CNN
+	1    3050 5700
 	1    0    0    -1
 $EndComp
@@
 L BMS_Hardware-rescue:R R2
 U 1 1 5BC607C0
-P 3450 5550
-F 0 "R2" H 3520 5596 50  0000 L CNN
-F 1 "36.5k" H 3520 5505 50  0000 L CNN
-F 2 "Resistor_SMD:R_0603_1608Metric_Pad1.05x0.95mm_HandSolder" V 3380 5550 50  0001 C CNN
-F 3 "" H 3450 5550 50  0001 C CNN
-	1    3450 5550
-	1    0    0    -1
-$EndComp
-Wire Wire Line
-	3150 5400 3450 5400
-Text GLabel 3550 5700 2    50   UnSpc ~ 0
-GND
-Wire Wire Line
-	2750 5700 3150 5700
-Connection ~ 2750 5700
+P 3350 5700
+F 0 "R2" H 3420 5746 50  0000 L CNN
+F 1 "36.5k" H 3420 5655 50  0000 L CNN
+F 2 "Resistor_SMD:R_0603_1608Metric_Pad1.05x0.95mm_HandSolder" V 3280 5700 50  0001 C CNN
+F 3 "" H 3350 5700 50  0001 C CNN
+	1    3350 5700
+	1    0    0    -1
+$EndComp
+Wire Wire Line
+	3050 5550 3350 5550
+Text GLabel 3450 5850 2    50   UnSpc ~ 0
+GND
+Wire Wire Line
+	2650 5850 3050 5850
+Connection ~ 2650 5850
 $Comp
 L BMS_Hardware-rescue:R R3
@@
 Wire Wire Line
 	2800 10150 3000 10150
-Text GLabel 3150 5050 0    50   Input ~ 0
+Text GLabel 3050 5200 0    50   Input ~ 0
 3V3
 $Comp
 L Device:D_Schottky D12
 U 1 1 5BCDE88D
-P 3150 5250
-F 0 "D12" V 3104 5329 50  0000 L CNN
-F 1 "D_Schottky" V 3195 5329 50  0000 L CNN
-F 2 "Diode_SMD:D_0603_1608Metric_Pad1.05x0.95mm_HandSolder" H 3150 5250 50  0001 C CNN
-F 3 "~" H 3150 5250 50  0001 C CNN
-	1    3150 5250
+P 3050 5400
+F 0 "D12" V 3004 5479 50  0000 L CNN
+F 1 "D_Schottky" V 3095 5479 50  0000 L CNN
+F 2 "Diode_SMD:D_0603_1608Metric_Pad1.05x0.95mm_HandSolder" H 3050 5400 50  0001 C CNN
+F 3 "~" H 3050 5400 50  0001 C CNN
+	1    3050 5400
 	0    1    1    0
 $EndComp
-Connection ~ 3150 5400
+Connection ~ 3050 5550
 Text GLabel 4750 5900 0    50   Input ~ 0
 3V3
@@
 Connection ~ 4750 6200
 Wire Wire Line
-	3450 5400 3700 5400
-Connection ~ 3450 5400
+	3350 5550 3600 5550
+Connection ~ 3350 5550
 Connection ~ 4750 6900
 Wire Wire Line
@@
 	11250 8700 11200 8700
 Wire Wire Line
-	3150 5100 3150 5050
+	3050 5250 3050 5200
 Wire Wire Line
 	4450 1750 4500 1750
@@
 	5050 6500 5150 6500
 Wire Wire Line
-	3550 5700 3450 5700
+	3450 5850 3350 5850
 Wire Wire Line
 	5150 8600 5050 8600

Commit message: started board edgecuts
Parts:
- Q6, Q7: footprint MRDT_ICs:IRLS3034_TO-263-7_P -> MRDT_Actives:IRLS3034_TO-263-7_P
- U16: footprint MRDT_Devices:OKI_Horisontal -> MRDT_Devices:OKI_Horizontal
Changed lines of the file:
@@
 F 0 "U16" H 11500 1050 60  0001 C CNN
 F 1 "OKI" H 11800 1650 60  0000 C CNN
-F 2 "MRDT_Devices:OKI_Horisontal" H 11400 1200 60  0001 C CNN
+F 2 "MRDT_Devices:OKI_Horizontal" H 11400 1200 60  0001 C CNN
 F 3 "" H 11400 1200 60  0001 C CNN
 	1    11650 1300
@@
 F 0 "Q7" H 7200 2325 50  0000 L CNN
 F 1 "IRLS3034-7P" H 7200 2250 50  0000 L CNN
-F 2 "MRDT_ICs:IRLS3034_TO-263-7_P" H 7200 2175 50  0001 L CIN
+F 2 "MRDT_Actives:IRLS3034_TO-263-7_P" H 7200 2175 50  0001 L CIN
 F 3 "" H 7000 2250 50  0001 L CNN
 	1    7000 2250
@@
 F 0 "Q6" H 6850 2825 50  0000 L CNN
 F 1 "IRLS3034-7P" H 6850 2750 50  0000 L CNN
-F 2 "MRDT_ICs:IRLS3034_TO-263-7_P" H 6850 2675 50  0001 L CIN
+F 2 "MRDT_Actives:IRLS3034_TO-263-7_P" H 6850 2675 50  0001 L CIN
 F 3 "" H 6650 2750 50  0001 L CNN
 	1    6650 2750
