File: BMS_Hardware/BMS_Hardware.kicad_pcb (KiCad board)
At the start: 2 copper layers, 208.3 x 76.2 mm, 131 parts, among them Q1 2N7002PW, Q2 2N7002PW, Q3 2N7002PW, Q4 2N7002PW, Q5 2N7002PW, Q6 IRLS3034-7P, Q7 IRLS3034-7P, Q8 2N7002PW, U1 ACS759ECB-200B-PFF-T, U10 E_STOP+LED, U11 TEMP, U12 FAN 4, U13 INA132, U14 INA132, U15 INA132, U16 OKI, U17 Indicator Comm, U18 OKI, U19 INA132, U2 FAN 1, U20 INA132, U21 TM4C129E_Launchpad, U3 INA132, U4 FAN 2, U5 Logic_Switch, U6 LT1910, U7 WIRELESS_E_STOP, U8 FAN 3, U9 INA132

Commit message: remade gerbs with new packaging
Parts:
- C10: footprint Capacitor_SMD:C_0603_1608Metric_Pad1.05x0.95mm_HandSolder -> Capacitor_SMD:C_1206_3216Metric_Pad1.42x1.75mm_HandSolder
- Conn2: value CHARGE SENSE -> CHARGE_SENSE_TOP
- D1, D12, D13, D2, D3, D4, D5, D6, D7, D8: footprint Diode_SMD:D_0603_1608Metric_Pad1.05x0.95mm_HandSolder -> Diode_SMD:D_SOD-323_HandSoldering
- U11: value TEMP -> TEMP_1
- U12: value FAN 4 -> FAN_4
- U2: value FAN 1 -> FAN_1
- U4: value FAN 2 -> FAN_2
- U5: value Logic_Switch -> BMS_Logic_Switch
- U7: value WIRELESS_E_STOP -> E_STOP
- U8: value FAN 3 -> FAN_3
- moved R13 93.2 mm to (174.6, 79.2), turned to 90 degrees
- moved U6 91.9 mm to (180.0, 78.2)
- moved C10 91.8 mm to (185.3, 77.9)
- moved R32 0.13 mm to (147.6, 105.8)
Connections:
- Conn3 pad 2: V_IN -> /V_IN
- Q6 pad 2: Net-(Q6-Pad2) -> Net-(C10-Pad1)
- Q7 pad 2: Net-(Q6-Pad2) -> Net-(C10-Pad1)
- U1 pad 5: Net-(Q6-Pad2) -> Net-(C10-Pad1)
- U5 pad 3: Net-(Q6-Pad2) -> Net-(C10-Pad1)
Routing:
- net V_IN: track 208.4 -> 0.00 mm
- net /V_IN: track 0.00 -> 208.4 mm
- net E-Stop_Gate: track 173.2 -> 69.0 mm, vias 2 -> 0
- net Net-(R13-Pad1): track 68.5 -> 157.5 mm, vias 2 -> 6
- net Net-(C10-Pad1): track 7.24 -> 49.8 mm, vias 0 -> 11
- net Net-(Q6-Pad2): track 31.4 -> 0.00 mm, vias 9 -> 0
- net GND: track 1.89 -> 1.92 mm, vias 122 -> 121
- added copper zone on B.Cu, net Net-(C10-Pad1)
- added copper zone on F.Cu, net Net-(C10-Pad1)
- removed copper zone on B.Cu, net Net-(Q6-Pad2)
- removed copper zone on F.Cu, net Net-(Q6-Pad2)

Commit message: updated ro KiCad libraries rev2
Parts:
- Conn3: footprint BMS_Hardware:Vertical Anderson Double -> MRDT_Connectors:Anderson_2_Horizontal_Stacked
- U1: footprint BMS_Hardware:PFF_Leadform_5pins -> MRDT_Sensors:ACS759ECB_PFF_Leadform_5pins
- U21: footprint BMS_Hardware:TM4C129E_Launchpad_FULL_Top_SMD -> MRDT_Shields:TM4C129E_Launchpad_FULL_SMD_TOP
Connections:
- C1 pad 2: CELL_1 -> (no net)
- C2 pad 2: LOGIC_PWR -> (no net)
- C26 pad 1: LOGIC_PWR -> (no net)
- C3 pad 2: LOGIC_PWR -> (no net)
- C4 pad 2: LOGIC_PWR -> (no net)
- C5 pad 2: LOGIC_PWR -> (no net)
- C6 pad 2: LOGIC_PWR -> (no net)
- C7 pad 2: LOGIC_PWR -> (no net)
- C8 pad 1: LOGIC_PWR -> (no net)
- D1 pad 1: CELL_1 -> (no net)
- D2 pad 1: CELL_8 -> (no net)
- R17 pad 1: CELL_8-7_SENSE -> (no net)
- R2 pad 1: CELL_1-GND_SENSE -> (no net)
- R21 pad 1: CELL_7-6_SENSE -> (no net)
- R30 pad 1: CELL_6-5_SENSE -> (no net)
- R31 pad 1: CELL_5-4_SENSE -> (no net)
- R32 pad 1: CELL_4-3_SENSE -> (no net)
- R33 pad 1: CELL_3-2_SENSE -> (no net)
- R34 pad 1: CELL_2-1_SENSE -> (no net)
- U13 pad 8: Net-(U13-Pad8) -> (no net)
- U14 pad 8: Net-(U14-Pad8) -> (no net)
- U15 pad 8: Net-(U15-Pad8) -> (no net)
- U19 pad 8: Net-(U19-Pad8) -> (no net)
- U20 pad 8: Net-(U20-Pad8) -> (no net)
- U21 pad +3V3: Net-(U21-Pad+3V3) -> (no net)
- U21 pad PA4: Net-(U21-PadPA4) -> (no net)
- U21 pad PA6: Net-(U21-PadPA6) -> (no net)
- U21 pad PA7: Net-(U21-PadPA7) -> (no net)
- U21 pad PB2: Net-(U21-PadPB2) -> (no net)
- U21 pad PB3: Net-(U21-PadPB3) -> (no net)
- U21 pad PC4: Net-(U21-PadPC4) -> (no net)
- U21 pad PC5: Net-(U21-PadPC5) -> (no net)
- U21 pad PC6: Net-(U21-PadPC6) -> (no net)
- U21 pad PC7: Net-(U21-PadPC7) -> (no net)
- U21 pad PD2: Net-(U21-PadPD2) -> (no net)
- U21 pad PD3: Net-(U21-PadPD3) -> (no net)
- U21 pad PD7: Net-(U21-PadPD7) -> (no net)
- U21 pad PE3: Net-(U21-PadPE3) -> (no net)
- U21 pad PE4: Net-(U21-PadPE4) -> (no net)
- U21 pad PE5: Net-(U21-PadPE5) -> (no net)
- U21 pad PF2: Net-(U21-PadPF2) -> (no net)
- U21 pad PF3: Net-(U21-PadPF3) -> (no net)
- U21 pad PG0: Net-(U21-PadPG0) -> (no net)
- U21 pad PG1: Net-(U21-PadPG1) -> (no net)
- U21 pad PH0: Net-(U21-PadPH0) -> (no net)
- U21 pad PH1: Net-(U21-PadPH1) -> (no net)
- U21 pad PK4: Net-(U21-PadPK4) -> (no net)
- U21 pad PK5: Net-(U21-PadPK5) -> (no net)
- U21 pad PK6: Net-(U21-PadPK6) -> (no net)
- U21 pad PK7: Net-(U21-PadPK7) -> (no net)
- U21 pad PL0: Net-(U21-PadPL0) -> (no net)
- U21 pad PL1: Net-(U21-PadPL1) -> (no net)
- U21 pad PL2: Net-(U21-PadPL2) -> (no net)
- U21 pad PL3: Net-(U21-PadPL3) -> (no net)
- U21 pad PM0: Net-(U21-PadPM0) -> (no net)
- U21 pad PM1: Net-(U21-PadPM1) -> (no net)
- U21 pad PM2: Net-(U21-PadPM2) -> (no net)
- U21 pad PM4: Net-(U21-PadPM4) -> (no net)
- U21 pad PM5: Net-(U21-PadPM5) -> (no net)
- U21 pad PM6: Net-(U21-PadPM6) -> (no net)
- U21 pad PM7: Net-(U21-PadPM7) -> (no net)
- U21 pad PN3: Net-(U21-PadPN3) -> (no net)
- U21 pad PN4: Net-(U21-PadPN4) -> (no net)
- U21 pad PN5: Net-(U21-PadPN5) -> (no net)
- U21 pad PP0: Net-(U21-PadPP0) -> (no net)
- U21 pad PP1: Net-(U21-PadPP1) -> (no net)
- U21 pad PP2: Net-(U21-PadPP2) -> (no net)
- U21 pad PP4: Net-(U21-PadPP4) -> (no net)
- U21 pad PP5: Net-(U21-PadPP5) -> (no net)
- U21 pad PQ0: Net-(U21-PadPQ0) -> (no net)
- U21 pad PQ1: Net-(U21-PadPQ1) -> (no net)
- U21 pad Rese: Net-(U21-PadRese) -> (no net)
- U3 pad 8: Net-(U3-Pad8) -> (no net)
- U6 pad 2: Net-(U6-Pad2) -> (no net)
- U6 pad 3: Net-(U6-Pad3) -> (no net)
- U9 pad 8: Net-(U9-Pad8) -> (no net)
Routing:
- net GND: track 1.92 -> 210.3 mm
- net /V_IN: track 208.4 -> 0.00 mm

Commit message: file problems fixed
Parts:
- added G***: LOGO, MRDT_Silkscreens:2_Dahlbot_2.0, F.Cu at (218.2, 77.7)
- Conn3: footprint MRDT_Connectors:Anderson_2_Horizontal_Stacked -> MRDT_Connectors:Anderson_2_Vertical_Sidy_by_Side
- D12, D13, D14, D15, D16, D17, D18, D19, D20, D22: value D_Schottky -> D_Zener
- R22: value 1M -> 100k
- R23: value 100k -> 10k
- R29: value 4.7k -> 820
- U12, U2, U4, U8: moved to B.Cu
- moved G*** 62.8 mm to (112.5, 65.5)
- moved D13 62.4 mm to (107.3, 85.7), turned to 270 degrees
- moved R29 55.4 mm to (87.5, 116.1)
- moved D17 39.4 mm to (145.8, 105.4)
- moved D20 23.1 mm to (168.4, 92.5), turned to 0 degrees
- moved Conn3 15.8 mm to (174.6, 53.6)
- moved D15 10.0 mm to (107.3, 105.3), turned to 270 degrees
- moved D14 9.65 mm to (107.3, 95.4), turned to 270 degrees
- moved D16 9.57 mm to (107.3, 114.7), turned to 270 degrees
- moved D19 8.89 mm to (145.8, 88.6), turned to 90 degrees
- moved D18 8.89 mm to (145.8, 97.2), turned to 90 degrees
- moved R15 5.70 mm to (168.0, 88.6), turned to 0 degrees
- moved R14 3.43 mm to (168.0, 90.4), turned to 180 degrees
- moved D22 3.27 mm to (87.9, 110.5), turned to 0 degrees
- moved R22 2.82 mm to (87.5, 112.5)
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Connections:
- C1 pad 2: (no net) -> CELL_1
- C2 pad 2: (no net) -> LOGIC_PWR
- C26 pad 1: (no net) -> LOGIC_PWR
- C3 pad 2: (no net) -> LOGIC_PWR
- C4 pad 2: (no net) -> LOGIC_PWR
- C5 pad 2: (no net) -> LOGIC_PWR
- C6 pad 2: (no net) -> LOGIC_PWR
- C7 pad 2: (no net) -> LOGIC_PWR
- C8 pad 1: (no net) -> LOGIC_PWR
- D1 pad 1: (no net) -> CELL_1
- D10 pad 2: PACK_V_IND -> V_OUT
- D12 pad 1: +3V3 -> CELL_1-GND_SENSE
- D12 pad 2: CELL_1-GND_SENSE -> GND
- D13 pad 1: +3V3 -> CELL_8-7_SENSE
- D13 pad 2: V_LOG_SENSE -> GND
- D14 pad 1: +3V3 -> CELL_7-6_SENSE
- D14 pad 2: CELL_8-7_SENSE -> GND
- D15 pad 1: +3V3 -> CELL_6-5_SENSE
- D15 pad 2: CELL_7-6_SENSE -> GND
- D16 pad 1: +3V3 -> CELL_5-4_SENSE
- D16 pad 2: CELL_6-5_SENSE -> GND
- D17 pad 1: +3V3 -> CELL_4-3_SENSE
- D17 pad 2: CELL_5-4_SENSE -> GND
- D18 pad 1: +3V3 -> CELL_3-2_SENSE
- D18 pad 2: CELL_4-3_SENSE -> GND
- D19 pad 1: +3V3 -> CELL_2-1_SENSE
- D19 pad 2: CELL_3-2_SENSE -> GND
- D2 pad 1: (no net) -> CELL_8
- D20 pad 1: +3V3 -> V_LOG_SENSE
- D20 pad 2: CELL_2-1_SENSE -> GND
- D22 pad 1: +3V3 -> V_OUT_SENSE
- D22 pad 2: V_OUT_SENSE -> GND
- R17 pad 1: (no net) -> CELL_8-7_SENSE
- R2 pad 1: (no net) -> CELL_1-GND_SENSE
- R21 pad 1: (no net) -> CELL_7-6_SENSE
- R23 pad 1: GND -> Net-(R23-Pad1)
- R29 pad 1: TEMP_D_OUT -> Net-(R23-Pad1)
- R30 pad 1: (no net) -> CELL_6-5_SENSE
- R31 pad 1: (no net) -> CELL_5-4_SENSE
- R32 pad 1: (no net) -> CELL_4-3_SENSE
- R33 pad 1: (no net) -> CELL_3-2_SENSE
- R34 pad 1: (no net) -> CELL_2-1_SENSE
- U13 pad 8: (no net) -> Net-(U13-Pad8)
- U14 pad 8: (no net) -> Net-(U14-Pad8)
- U15 pad 8: (no net) -> Net-(U15-Pad8)
- U19 pad 8: (no net) -> Net-(U19-Pad8)
- U20 pad 8: (no net) -> Net-(U20-Pad8)
- U21 pad +3V3: (no net) -> Net-(U21-Pad+3V3)
- U21 pad PA4: (no net) -> Net-(U21-PadPA4)
- U21 pad PA6: (no net) -> Net-(U21-PadPA6)
- U21 pad PA7: (no net) -> Net-(U21-PadPA7)
- U21 pad PB2: (no net) -> Net-(U21-PadPB2)
- U21 pad PB3: (no net) -> Net-(U21-PadPB3)
- U21 pad PC4: (no net) -> Net-(U21-PadPC4)
- U21 pad PC5: (no net) -> Net-(U21-PadPC5)
- U21 pad PC6: (no net) -> Net-(U21-PadPC6)
- U21 pad PC7: (no net) -> Net-(U21-PadPC7)
- U21 pad PD0: LOGIC_SWITCH -> Net-(U21-PadPD0)
- U21 pad PD1: PACK_GATE -> TEMP_D_OUT
- U21 pad PD2: (no net) -> Net-(U21-PadPD2)
- U21 pad PD3: (no net) -> Net-(U21-PadPD3)
- U21 pad PD7: (no net) -> Net-(U21-PadPD7)
- U21 pad PE3: (no net) -> Net-(U21-PadPE3)
- U21 pad PE4: (no net) -> Net-(U21-PadPE4)
- U21 pad PE5: (no net) -> Net-(U21-PadPE5)
- U21 pad PF2: (no net) -> Net-(U21-PadPF2)
- U21 pad PF3: (no net) -> Net-(U21-PadPF3)
- U21 pad PG0: (no net) -> Net-(U21-PadPG0)
- U21 pad PG1: (no net) -> Net-(U21-PadPG1)
- U21 pad PH0: (no net) -> Net-(U21-PadPH0)
- U21 pad PH1: (no net) -> Net-(U21-PadPH1)
- U21 pad PK4: (no net) -> Net-(U21-PadPK4)
- U21 pad PK5: (no net) -> Net-(U21-PadPK5)
- U21 pad PK6: (no net) -> Net-(U21-PadPK6)
- U21 pad PK7: (no net) -> Net-(U21-PadPK7)
- U21 pad PL0: (no net) -> Net-(U21-PadPL0)
- U21 pad PL1: (no net) -> Net-(U21-PadPL1)
- U21 pad PL2: (no net) -> Net-(U21-PadPL2)
- U21 pad PL3: (no net) -> Net-(U21-PadPL3)
- U21 pad PM0: (no net) -> Net-(U21-PadPM0)
- U21 pad PM1: (no net) -> Net-(U21-PadPM1)
- U21 pad PM2: (no net) -> Net-(U21-PadPM2)
- U21 pad PM3: TEMP_D_OUT -> Net-(U21-PadPM3)
- U21 pad PM4: (no net) -> Net-(U21-PadPM4)
- U21 pad PM5: (no net) -> Net-(U21-PadPM5)
- U21 pad PM6: (no net) -> Net-(U21-PadPM6)
- U21 pad PM7: (no net) -> Net-(U21-PadPM7)
- U21 pad PN3: (no net) -> PACK_GATE
- U21 pad PN4: (no net) -> Net-(U21-PadPN4)
- U21 pad PN5: (no net) -> Net-(U21-PadPN5)
- U21 pad PP0: (no net) -> Net-(U21-PadPP0)
- U21 pad PP1: (no net) -> Net-(U21-PadPP1)
- U21 pad PP2: (no net) -> LOGIC_SWITCH
- U21 pad PP4: (no net) -> Net-(U21-PadPP4)
- U21 pad PP5: (no net) -> Net-(U21-PadPP5)
- U21 pad PQ0: (no net) -> Net-(U21-PadPQ0)
- U21 pad PQ1: (no net) -> Net-(U21-PadPQ1)
- U21 pad PQ2: PACK_V_IND -> Net-(U21-PadPQ2)
- U21 pad Rese: (no net) -> Net-(U21-PadRese)
- U21 pad Rese': (no net) -> Net-(U21-PadRese')
- U3 pad 8: (no net) -> Net-(U3-Pad8)
- U6 pad 2: (no net) -> Net-(U6-Pad2)
- U6 pad 3: (no net) -> Net-(U6-Pad3)
- U9 pad 8: (no net) -> Net-(U9-Pad8)
Routing:
- net +3V3: track 435.2 -> 174.1 mm, vias 13 -> 2
- net /V_IN: track 0.00 -> 212.2 mm, vias 30 -> 31
- net GND: track 210.3 -> 1.92 mm, vias 121 -> 117
- net PACK_V_IND: track 66.3 -> 0.00 mm, vias 2 -> 0
- net V_OUT: track 180.5 -> 226.3 mm, vias 30 -> 32
- net Net-(R13-Pad1): track 157.5 -> 147.0 mm
- net PACK_GATE: track 38.1 -> 45.7 mm
- net TEMP_D_OUT: track 47.7 -> 40.3 mm, vias 2 -> 0
- net LOGIC_PWR: track 288.1 -> 292.8 mm
- net LOGIC_SWITCH: track 19.9 -> 16.4 mm
- net V_OUT_SENSE: track 12.9 -> 15.0 mm
- net CELL_1: track 77.0 -> 79.1 mm
- net CELL_2-1_SENSE: track 42.0 -> 40.1 mm
- net Net-(R23-Pad1): track 0.00 -> 1.78 mm
- net V_LOG_SENSE: track 122.8 -> 121.6 mm
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Other:
- board text added: "BMS, REV. 2 MARS ROVER DESIGN TEAM MISSOURI S&T, 2019 Brian Dahlman"
- board text removed: "BMS, REV. 1 MARS ROVER DESIGN TEAM MISSOURI S&T, 2019"
