File: BMS_Hardware/BMS_Hardware.sch (KiCad schematic (older format))
At the start: 123 parts, among them Q1 2N7002PW, Q2 2N7002PW, Q3 2N7002PW, Q4 2N7002PW, Q5 2N7002PW, Q6 IRLS3034-7P, Q7 IRLS3034-7P, Q8 2N7002PW, U1 ACS759ECB-200B-PFF-T, U10 E_STOP+LED, U11 TEMP_1, U12 FAN_4, U13 INA132, U14 INA132, U15 INA132, U16 OKI, U17 Indicator Comm, U18 OKI, U19 INA132, U2 FAN_1, U20 INA132, U21 TM4C129E_Launchpad, U3 INA132, U4 FAN_2, U5 BMS_Logic_Switch, U6 LT1910, U7 E_STOP, U8 FAN_3, U9 INA132

Commit message: final changes to layout
Connections:
- wire segments 394 -> 434

Commit message: changed footprints of schottkey diode
Parts:
- D1, D2, D3, D4, D5, D6, D7, D8: footprint Diode_SMD:D_0603_1608Metric_Pad1.05x0.95mm_HandSolder -> Diode_SMD:D_SOD-323_HandSoldering
Changed lines of the file:
@@
 F 0 "D1" H 3800 12250 50  0000 C CNN
 F 1 "7.5V" H 3800 12050 50  0000 C CNN
-F 2 "Diode_SMD:D_0603_1608Metric_Pad1.05x0.95mm_HandSolder" H 3800 12150 50  0001 C CNN
+F 2 "Diode_SMD:D_SOD-323_HandSoldering" H 3800 12150 50  0001 C CNN
 F 3 "" H 3800 12150 50  0001 C CNN
 	1    3800 12150
@@
 F 0 "D2" H 2750 5700 50  0000 C CNN
 F 1 "7.5V" H 2750 5500 50  0000 C CNN
-F 2 "Diode_SMD:D_0603_1608Metric_Pad1.05x0.95mm_HandSolder" H 2750 5600 50  0001 C CNN
+F 2 "Diode_SMD:D_SOD-323_HandSoldering" H 2750 5600 50  0001 C CNN
 F 3 "" H 2750 5600 50  0001 C CNN
 	1    2750 5600
@@
 F 0 "D3" H 2750 6600 50  0000 C CNN
 F 1 "7.5V" H 2750 6400 50  0000 C CNN
-F 2 "Diode_SMD:D_0603_1608Metric_Pad1.05x0.95mm_HandSolder" H 2750 6500 50  0001 C CNN
+F 2 "Diode_SMD:D_SOD-323_HandSoldering" H 2750 6500 50  0001 C CNN
 F 3 "" H 2750 6500 50  0001 C CNN
 	1    2750 6500
@@
 F 0 "D4" H 2750 7500 50  0000 C CNN
 F 1 "7.5V" H 2750 7300 50  0000 C CNN
-F 2 "Diode_SMD:D_0603_1608Metric_Pad1.05x0.95mm_HandSolder" H 2750 7400 50  0001 C CNN
+F 2 "Diode_SMD:D_SOD-323_HandSoldering" H 2750 7400 50  0001 C CNN
 F 3 "" H 2750 7400 50  0001 C CNN
 	1    2750 7400
@@
 F 0 "D5" H 2750 8400 50  0000 C CNN
 F 1 "7.5V" H 2750 8200 50  0000 C CNN
-F 2 "Diode_SMD:D_0603_1608Metric_Pad1.05x0.95mm_HandSolder" H 2750 8300 50  0001 C CNN
+F 2 "Diode_SMD:D_SOD-323_HandSoldering" H 2750 8300 50  0001 C CNN
 F 3 "" H 2750 8300 50  0001 C CNN
 	1    2750 8300
@@
 F 0 "D6" H 2750 9300 50  0000 C CNN
 F 1 "7.5V" H 2750 9100 50  0000 C CNN
-F 2 "Diode_SMD:D_0603_1608Metric_Pad1.05x0.95mm_HandSolder" H 2750 9200 50  0001 C CNN
+F 2 "Diode_SMD:D_SOD-323_HandSoldering" H 2750 9200 50  0001 C CNN
 F 3 "" H 2750 9200 50  0001 C CNN
 	1    2750 9200
@@
 F 0 "D7" H 2750 10200 50  0000 C CNN
 F 1 "7.5V" H 2750 10000 50  0000 C CNN
-F 2 "Diode_SMD:D_0603_1608Metric_Pad1.05x0.95mm_HandSolder" H 2750 10100 50  0001 C CNN
+F 2 "Diode_SMD:D_SOD-323_HandSoldering" H 2750 10100 50  0001 C CNN
 F 3 "" H 2750 10100 50  0001 C CNN
 	1    2750 10100
@@
 F 0 "D8" H 2750 11100 50  0000 C CNN
 F 1 "7.5V" H 2750 10900 50  0000 C CNN
-F 2 "Diode_SMD:D_0603_1608Metric_Pad1.05x0.95mm_HandSolder" H 2750 11000 50  0001 C CNN
+F 2 "Diode_SMD:D_SOD-323_HandSoldering" H 2750 11000 50  0001 C CNN
 F 3 "" H 2750 11000 50  0001 C CNN
 	1    2750 11000

Commit message: remade gerbs with new packaging
Parts:
- C10: footprint Capacitor_SMD:C_0603_1608Metric_Pad1.05x0.95mm_HandSolder -> Capacitor_SMD:C_1206_3216Metric_Pad1.42x1.75mm_HandSolder
- D12, D13, D14, D15, D16, D17, D18, D19, D20, D22: footprint Diode_SMD:D_0603_1608Metric_Pad1.05x0.95mm_HandSolder -> Diode_SMD:D_SOD-323_HandSoldering
Connections:
- wire segments 434 -> 437
Changed lines of the file:
@@
 F 0 "C10" H 5060 3470 50  0000 L CNN
 F 1 "10u" H 5060 3320 50  0000 L CNN
-F 2 "Capacitor_SMD:C_0603_1608Metric_Pad1.05x0.95mm_HandSolder" H 5050 3400 50  0001 C CNN
+F 2 "Capacitor_SMD:C_1206_3216Metric_Pad1.42x1.75mm_HandSolder" H 5050 3400 50  0001 C CNN
 F 3 "" H 5050 3400 50  0001 C CNN
 	1    5050 3400
@@
 F 0 "D12" V 4354 11929 50  0000 L CNN
 F 1 "D_Schottky" V 4445 11929 50  0000 L CNN
-F 2 "Diode_SMD:D_0603_1608Metric_Pad1.05x0.95mm_HandSolder" H 4400 11850 50  0001 C CNN
+F 2 "Diode_SMD:D_SOD-323_HandSoldering" H 4400 11850 50  0001 C CNN
 F 3 "~" H 4400 11850 50  0001 C CNN
 	1    4400 11850
@@
 F 0 "D14" H 4700 5550 50  0000 L CNN
 F 1 "D_Schottky" H 4650 5350 50  0000 L CNN
-F 2 "Diode_SMD:D_0603_1608Metric_Pad1.05x0.95mm_HandSolder" H 4800 5450 50  0001 C CNN
+F 2 "Diode_SMD:D_SOD-323_HandSoldering" H 4800 5450 50  0001 C CNN
 F 3 "~" H 4800 5450 50  0001 C CNN
 	1    4800 5450
@@
 F 0 "D15" H 4700 6450 50  0000 L CNN
 F 1 "D_Schottky" H 4650 6250 50  0000 L CNN
-F 2 "Diode_SMD:D_0603_1608Metric_Pad1.05x0.95mm_HandSolder" H 4800 6350 50  0001 C CNN
+F 2 "Diode_SMD:D_SOD-323_HandSoldering" H 4800 6350 50  0001 C CNN
 F 3 "~" H 4800 6350 50  0001 C CNN
 	1    4800 6350
@@
 F 0 "D16" H 4700 7350 50  0000 L CNN
 F 1 "D_Schottky" H 4650 7150 50  0000 L CNN
-F 2 "Diode_SMD:D_0603_1608Metric_Pad1.05x0.95mm_HandSolder" H 4800 7250 50  0001 C CNN
+F 2 "Diode_SMD:D_SOD-323_HandSoldering" H 4800 7250 50  0001 C CNN
 F 3 "~" H 4800 7250 50  0001 C CNN
 	1    4800 7250
@@
 F 0 "D17" H 4700 8250 50  0000 L CNN
 F 1 "D_Schottky" H 4650 8050 50  0000 L CNN
-F 2 "Diode_SMD:D_0603_1608Metric_Pad1.05x0.95mm_HandSolder" H 4800 8150 50  0001 C CNN
+F 2 "Diode_SMD:D_SOD-323_HandSoldering" H 4800 8150 50  0001 C CNN
 F 3 "~" H 4800 8150 50  0001 C CNN
 	1    4800 8150
@@
 F 0 "D18" H 4754 9129 50  0000 L CNN
 F 1 "D_Schottky" H 4700 8950 50  0000 L CNN
-F 2 "Diode_SMD:D_0603_1608Metric_Pad1.05x0.95mm_HandSolder" H 4800 9050 50  0001 C CNN
+F 2 "Diode_SMD:D_SOD-323_HandSoldering" H 4800 9050 50  0001 C CNN
 F 3 "~" H 4800 9050 50  0001 C CNN
 	1    4800 9050
@@
 F 0 "D19" H 4750 10050 50  0000 L CNN
 F 1 "D_Schottky" H 4650 9850 50  0000 L CNN
-F 2 "Diode_SMD:D_0603_1608Metric_Pad1.05x0.95mm_HandSolder" H 4800 9950 50  0001 C CNN
+F 2 "Diode_SMD:D_SOD-323_HandSoldering" H 4800 9950 50  0001 C CNN
 F 3 "~" H 4800 9950 50  0001 C CNN
 	1    4800 9950
@@
 F 0 "D20" H 4750 10950 50  0000 L CNN
 F 1 "D_Schottky" H 4650 10750 50  0000 L CNN
-F 2 "Diode_SMD:D_0603_1608Metric_Pad1.05x0.95mm_HandSolder" H 4800 10850 50  0001 C CNN
+F 2 "Diode_SMD:D_SOD-323_HandSoldering" H 4800 10850 50  0001 C CNN
 F 3 "~" H 4800 10850 50  0001 C CNN
 	1    4800 10850
@@
 F 0 "D22" V 9396 3121 50  0000 R CNN
 F 1 "D_Schottky" H 9305 3121 50  0000 R CNN
-F 2 "Diode_SMD:D_0603_1608Metric_Pad1.05x0.95mm_HandSolder" H 9350 3200 50  0001 C CNN
+F 2 "Diode_SMD:D_SOD-323_HandSoldering" H 9350 3200 50  0001 C CNN
 F 3 "~" H 9350 3200 50  0001 C CNN
 	1    9350 3200
@@
 F 0 "D13" V 7096 1771 50  0000 R CNN
 F 1 "D_Schottky" H 7005 1771 50  0000 R CNN
-F 2 "Diode_SMD:D_0603_1608Metric_Pad1.05x0.95mm_HandSolder" H 7050 1850 50  0001 C CNN
+F 2 "Diode_SMD:D_SOD-323_HandSoldering" H 7050 1850 50  0001 C CNN
 F 3 "~" H 7050 1850 50  0001 C CNN
 	1    7050 1850
@@
 $EndComp
 Wire Wire Line
-	3700 2650 6450 2650
+	3700 2650 5300 2650
 Wire Wire Line
 	5650 3650 5600 3650
 Wire Wire Line
-	5050 3150 5550 3150
+	5050 3150 5300 3150
 Wire Wire Line
 	5050 4150 6200 4150
@@
 Wire Wire Line
 	13550 3450 13550 3500
+Wire Wire Line
+	5300 2650 5300 3150
+Connection ~ 5300 2650
+Wire Wire Line
+	5300 2650 6450 2650
+Connection ~ 5300 3150
+Wire Wire Line
+	5300 3150 5550 3150
 $EndSCHEMATC

Commit message: updated ro KiCad libraries rev2
Parts:
- B1: symbol BMS_Hardware-rescue:BUZZER_SMI_1324_TW_5V_2_R -> MRDT_Devices:Buzzer
- C1, C10, C11, C12, C13, C14, C15, C16, C18, C19, C2, C20, C21, C22, C27, C28, C29, C3, C30, C31, C4, C5, C6, C7, C8, C9: symbol BMS_Hardware-rescue:C -> Device:C
- C17, C26: symbol BMS_Hardware-rescue:CP1 -> Device:CP1
- Conn1, Conn2: symbol BMS_Hardware-rescue:Molex_SL_9 -> MRDT_Connectors:Molex_SL_09
- Conn3: footprint BMS_Hardware:Vertical Anderson Double -> MRDT_Connectors:Anderson_2_Horizontal_Stacked
- D1, D2, D3, D4, D5, D6, D7, D8: symbol BMS_Hardware-rescue:D_Zener -> Device:D_Zener
- D10, D11, D21, D23, D9: symbol BMS_Hardware-rescue:LED -> Device:LED
- F1: symbol BMS_Hardware-rescue:Polyfuse -> Device:Polyfuse
- Q1, Q2, Q3, Q4, Q5, Q8: symbol BMS_Hardware-rescue:2N7002 -> Transistor_FET:2N7002
- R1, R10, R11, R12, R13, R14, R15, R16, R17, R18, R19, R2, R20, R21, R22, R23, R24, R25, R26, R27, R28, R29, R3, R30, R31, R32, R33, R34, R35, R4, R5, R6, R7, R8, R9: symbol BMS_Hardware-rescue:R -> Device:R
- U1: footprint BMS_Hardware:PFF_Leadform_5pins -> MRDT_Sensors:ACS759ECB_PFF_Leadform_5pins; symbol BMS_Hardware-rescue:ACS759ECB-200B-PFF-T -> MRDT_Sensors:ACS759ECB-200B-PFF-T
- U10: symbol BMS_Hardware-rescue:Molex_SL_4 -> MRDT_Connectors:Molex_SL_04
- U11, U17: symbol BMS_Hardware-rescue:Molex_SL_3 -> MRDT_Connectors:Molex_SL_03
- U12, U2, U4, U7, U8: symbol BMS_Hardware-rescue:Molex_SL_2 -> MRDT_Connectors:Molex_SL_02
- U16, U18: symbol BMS_Hardware-rescue:OKI -> MRDT_Devices:OKI
- U21: footprint BMS_Hardware:TM4C129E_Launchpad_FULL_Top_SMD -> MRDT_Shields:TM4C129E_Launchpad_FULL_SMD_TOP
- U5: symbol BMS_Logic_Switch:BMS_Logic_Switch -> MRDT_Switches:Relay_SPST
- U6: symbol BMS_Hardware-rescue:LT1910 -> MRDT_ICs:LT1910
- V1, V2, V3: symbol BMS_Hardware-rescue:BATT_PWR_VIA -> MRDT_Drill_Holes:BATT_PWR_VIA
Connections:
- wire segments 437 -> 414
- no-connect marks 60 -> 59

Commit message: file problems fixed
Parts:
- removed D12, D13, D14, D15, D16, D17, D18, D19, D20, D22: D_Schottky, Diode_SMD:D_SOD-323_HandSoldering, symbol Device:D_Schottky
- added D12, D13, D14, D15, D16, D17, D18, D19, D20, D22: D_Zener, Diode_SMD:D_SOD-323_HandSoldering, symbol Device:D_Zener
- Conn3: footprint MRDT_Connectors:Anderson_2_Horizontal_Stacked -> MRDT_Connectors:Anderson_2_Vertical_Sidy_by_Side
- R22: value 1M -> 100k
- R23: value 100k -> 10k
- R29: value 4.7k -> 820
Connections:
- net labels removed: PACK_V_IND
- wire segments 414 -> 449
- no-connect marks 59 -> 60
Other:
- note removed: "A15"
- moved on the sheet: C1, C2, C3, C4, C5, C6, C7, C8, D1, D2, D23, R17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
