File: BMS_Hardware/2020_BMSBOARD.kicad_pcb (KiCad board)
At the start: 2 copper layers, 137 parts, among them Q1 2N7002, Q2 Q_NMOS_GDS, Q3 Device_Q_NMOS_GDS, Q4 2N7002PW, Q5 2N7002PW, Q6 2N7002PW, Q7 2N7002PW, Q8 2N7002PW, SW1 Relay_SPST-MRDT_Switches, U1 LT1910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

Commit message: ok
Parts:
- moved R27 126.1 mm to (210.3, -38.2)
- moved R28 115.7 mm to (210.3, -41.1)
- moved R14 95.3 mm to (210.3, -44.1), turned to 180 degrees
- moved R35 94.7 mm to (215.6, -48.5)
- moved D17 57.8 mm to (210.3, -35.2)
- moved R13 2.59 mm to (210.2, -46.9), turned to 180 degrees
Changed lines of the file:
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@@
   )
   (module LED_SMD:LED_0603_1608Metric_Pad1.05x0.95mm_HandSolder (layer F.Cu)
-    (at 246.575001 9.775001)
+    (at 210.312 -35.179)
     (descr "LED SMD 0603 (1608 Metric), square (rectangular) end terminal, IPC_7351 nominal, (Body size source: http://www.tortai-tech.com/upload/download/2011102023233369053.pdf), generated with kicad-footprint-generator")
     (tags "LED handsolder")
     (attr smd)
-    (fp_text reference D17 (at 0 -1.43) (layer F.SilkS)
+    (fp_text reference D17 (at 0 1.524) (layer F.SilkS)
       (effects (font (size 1 1) (thickness 0.15)))
     )
@@
   )
   (module Resistor_SMD:R_0603_1608Metric_Pad1.05x0.95mm_HandSolder (layer F.Cu)
-    (at 210.693 -44.323)
+    (at 210.185 -46.863 180)
     (descr "Resistor SMD 0603 (1608 Metric), square (rectangular) end terminal, IPC_7351 nominal with elongated pad for handsoldering. (Body size source: http://www.tortai-tech.com/upload/download/2011102023233369053.pdf), generated with kicad-footprint-generator")
     (tags "resistor handsolder")
@@
     (fp_line (start -0.8 -0.4) (end 0.8 -0.4) (layer F.Fab) (width 0.1))
     (fp_line (start -0.8 0.4) (end -0.8 -0.4) (layer F.Fab) (width 0.1))
-    (pad 2 smd roundrect (at 0.875 0) (size 1.05 0.95) (layers F.Cu F.Paste F.Mask) (roundrect_rratio 0.25)
+    (pad 2 smd roundrect (at 0.875 0 180) (size 1.05 0.95) (layers F.Cu F.Paste F.Mask) (roundrect_rratio 0.25)
       (net 11 CELL_2))
-    (pad 1 smd roundrect (at -0.875 0) (size 1.05 0.95) (layers F.Cu F.Paste F.Mask) (roundrect_rratio 0.25)
+    (pad 1 smd roundrect (at -0.875 0 180) (size 1.05 0.95) (layers F.Cu F.Paste F.Mask) (roundrect_rratio 0.25)
       (net 65 "Net-(R13-Pad1)"))
     (model ${KISYS3DMOD}/Resistor_SMD.3dshapes/R_0603_1608Metric.wrl
@@
   )
   (module Resistor_SMD:R_0603_1608Metric_Pad1.05x0.95mm_HandSolder (layer F.Cu)
-    (at 254.290001 40.505001)
-    (descr "Resistor SMD 0603 (1608 Metric), square (rectangular) end terminal, IPC_7351 nominal with elongated pad for handsoldering. (Body size source: http://www.tortai-tech.com/upload/download/2011102023233369053.pdf), generated with kicad-footprint-generator")
-    (tags "resistor handsolder")
-    (attr smd)
-    (fp_text reference R14 (at 0 -1.43) (layer F.SilkS)
-      (effects (font (size 1 1) (thickness 0.15)))
-    )
-    (fp_text value R (at 0 1.43) (layer F.Fab)
-      (effects (font (size 1 1) (thickness 0.15)))
-    )
-    (fp_line (start -0.8 0.4) (end -0.8 -0.4) (layer F.Fab) (width 0.1))
-    (fp_line (start -0.8 -0.4) (end 0.8 -0.4) (layer F.Fab) (width 0.1))
-    (fp_line (start 0.8 -0.4) (end 0.8 0.4) (layer F.Fab) (width 0.1))
-    (fp_line (start 0.8 0.4) (end -0.8 0.4) (layer F.Fab) (width 0.1))
-    (fp_line (start -0.171267 -0.51) (end 0.171267 -0.51) (layer F.SilkS) (width 0.12))
-    (fp_line (start -0.171267 0.51) (end 0.171267 0.51) (layer F.SilkS) (width 0.12))
-    (fp_line (start -1.65 0.73) (end -1.65 -0.73) (layer F.CrtYd) (width 0.05))
-    (fp_line (start -1.65 -0.73) (end 1.65 -0.73) (layer F.CrtYd) (width 0.05))
-    (fp_line (start 1.65 -0.73) (end 1.65 0.73) (layer F.CrtYd) (width 0.05))
-    (fp_line (start 1.65 0.73) (end -1.65 0.73) (layer F.CrtYd) (width 0.05))
-    (fp_text user %R (at 0 0) (layer F.Fab)
-      (effects (font (size 0.4 0.4) (thickness 0.06)))
-    )
-    (pad 1 smd roundrect (at -0.875 0) (size 1.05 0.95) (layers F.Cu F.Paste F.Mask) (roundrect_rratio 0.25)
+    (at 210.312 -44.069 180)
+    (descr "Resistor SMD 0603 (1608 Metric), square (rectangular) end terminal, IPC_7351 nominal with elongated pad for handsoldering. (Body size source: http://www.tortai-tech.com/upload/download/2011102023233369053.pdf), generated with kicad-footprint-generator")
+    (tags "resistor handsolder")
+    (attr smd)
+    (fp_text reference R14 (at 0 -4.318) (layer F.SilkS)
+      (effects (font (size 1 1) (thickness 0.15)))
+    )
+    (fp_text value R (at 0 1.43) (layer F.Fab)
+      (effects (font (size 1 1) (thickness 0.15)))
+    )
+    (fp_line (start -0.8 0.4) (end -0.8 -0.4) (layer F.Fab) (width 0.1))
+    (fp_line (start -0.8 -0.4) (end 0.8 -0.4) (layer F.Fab) (width 0.1))
+    (fp_line (start 0.8 -0.4) (end 0.8 0.4) (layer F.Fab) (width 0.1))
+    (fp_line (start 0.8 0.4) (end -0.8 0.4) (layer F.Fab) (width 0.1))
+    (fp_line (start -0.171267 -0.51) (end 0.171267 -0.51) (layer F.SilkS) (width 0.12))
+    (fp_line (start -0.171267 0.51) (end 0.171267 0.51) (layer F.SilkS) (width 0.12))
+    (fp_line (start -1.65 0.73) (end -1.65 -0.73) (layer F.CrtYd) (width 0.05))
+    (fp_line (start -1.65 -0.73) (end 1.65 -0.73) (layer F.CrtYd) (width 0.05))
+    (fp_line (start 1.65 -0.73) (end 1.65 0.73) (layer F.CrtYd) (width 0.05))
+    (fp_line (start 1.65 0.73) (end -1.65 0.73) (layer F.CrtYd) (width 0.05))
+    (fp_text user %R (at 0 0) (layer F.Fab)
+      (effects (font (size 0.4 0.4) (thickness 0.06)))
+    )
+    (pad 1 smd roundrect (at -0.875 0 180) (size 1.05 0.95) (layers F.Cu F.Paste F.Mask) (roundrect_rratio 0.25)
       (net 66 "Net-(R14-Pad1)"))
-    (pad 2 smd roundrect (at 0.875 0) (size 1.05 0.95) (layers F.Cu F.Paste F.Mask) (roundrect_rratio 0.25)
+    (pad 2 smd roundrect (at 0.875 0 180) (size 1.05 0.95) (layers F.Cu F.Paste F.Mask) (roundrect_rratio 0.25)
       (net 12 CELL_1))
     (model ${KISYS3DMOD}/Resistor_SMD.3dshapes/R_0603_1608Metric.wrl
@@
   )
   (module Resistor_SMD:R_0603_1608Metric_Pad1.05x0.95mm_HandSolder (layer F.Cu)
-    (at 211.480001 87.845001)
-    (descr "Resistor SMD 0603 (1608 Metric), square (rectangular) end terminal, IPC_7351 nominal with elongated pad for handsoldering. (Body size source: http://www.tortai-tech.com/upload/download/2011102023233369053.pdf), generated with kicad-footprint-generator")
-    (tags "resistor handsolder")
-    (attr smd)
-    (fp_text reference R27 (at 0 -1.43) (layer F.SilkS)
+    (at 210.312 -38.227)
+    (descr "Resistor SMD 0603 (1608 Metric), square (rectangular) end terminal, IPC_7351 nominal with elongated pad for handsoldering. (Body size source: http://www.tortai-tech.com/upload/download/2011102023233369053.pdf), generated with kicad-footprint-generator")
+    (tags "resistor handsolder")
+    (attr smd)
+    (fp_text reference R27 (at -0.014 1.524) (layer F.SilkS)
       (effects (font (size 1 1) (thickness 0.15)))
     )
@@
   )
   (module Resistor_SMD:R_0603_1608Metric_Pad1.05x0.95mm_HandSolder (layer F.Cu)
-    (at 226.110001 73.515001)
+    (at 210.298 -41.148)
     (descr "Resistor SMD 0603 (1608 Metric), square (rectangular) end terminal, IPC_7351 nominal with elongated pad for handsoldering. (Body size source: http://www.tortai-tech.com/upload/download/2011102023233369053.pdf), generated with kicad-footprint-generator")
     (tags "resistor handsolder")
@@
   )
   (module Resistor_SMD:R_0603_1608Metric_Pad1.05x0.95mm_HandSolder (layer F.Cu)
-    (at 254.290001 37.995001)
-    (descr "Resistor SMD 0603 (1608 Metric), square (rectangular) end terminal, IPC_7351 nominal with elongated pad for handsoldering. (Body size source: http://www.tortai-tech.com/upload/download/2011102023233369053.pdf), generated with kicad-footprint-generator")
-    (tags "resistor handsolder")
+    (at 215.646 -48.514)
+    (descr "Resistor SMD 0603 (1608 Metric), square (rectangular) end terminal, IPC_7351 nominal with elongated pad for handsoldering. (Body size source: http://www.tortai-tech.com/upload/download/2011102023233369053.pdf), generated with kicad-footprint-generator")
+    (tags "resistor handsolder")

Commit message: updated layout
Parts:
- R1, R10, R11, R12, R13, R14, R2, R3, R4, R5, R6, R7, R8, R9: value R -> 6.65M
- R15, R16, R17, R18, R19, R20, R21, R22, R23, R24, R25, R26, R27, R28: value R -> 3.32M
- R32, R33, R34, R35, R36, R37, R38: value R -> 10k
- moved Q8 233.6 mm to (50.0, 2.03), turned to 270 degrees
- moved R54 224.7 mm to (50.0, -10.4)
- moved R30 223.1 mm to (60.2, -18.9), turned to 90 degrees
- moved Conn5 222.5 mm to (42.9, -24.8)
- moved Conn7 220.5 mm to (43.1, -7.62)
- moved Conn2 211.4 mm to (59.8, -8.38)
- moved R53 210.1 mm to (49.7, -27.6)
- moved Conn8 208.5 mm to (42.9, 1.14)
- moved R40 204.7 mm to (67.1, -19.1), turned to 90 degrees
- moved Q5 203.8 mm to (49.8, -24.0), turned to 270 degrees
- moved Conn6 203.0 mm to (42.9, -16.1)
- moved Q7 202.8 mm to (50.0, -15.4), turned to 270 degrees
- moved R39 202.3 mm to (63.8, -18.9), turned to 90 degrees
- moved R56 190.1 mm to (49.9, -1.65)
- moved R55 181.9 mm to (50.0, -19.3)
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Connections:
- net Net-(Conn1-Pad4) renamed V_IN

Commit message: almost done
Parts:
- moved R26 239.9 mm to (43.1, 32.0)
- moved R11 232.3 mm to (43.1, 27.7)
- moved R25 232.1 mm to (43.2, 25.8)
- moved R9 220.7 mm to (62.4, 28.1)
- moved R34 219.9 mm to (43.1, 34.2)
- moved R24 217.7 mm to (62.4, 33.3)
- moved R12 215.7 mm to (43.1, 29.8)
- moved R10 213.2 mm to (62.3, 30.8)
- moved V1 204.7 mm to (53.4, 45.6)
- moved R3 201.6 mm to (81.9, 26.9)
- moved D7 197.9 mm to (50.0, 22.0)
- moved R23 196.7 mm to (62.4, 26.0)
- moved R17 193.5 mm to (81.9, 28.8)
- moved R21 193.0 mm to (62.4, 12.6)
- moved R35 184.9 mm to (43.0, 17.5)
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Connections:
- Conn1 pad 2: (no net) -> V_IN
Routing:
- net V_IN: track 0.00 -> 211.2 mm, vias 0 -> 1
- net Net-(R27-Pad2): track 0.00 -> 1.49 mm
- added copper zone on B.Cu, net V_IN
- added copper zone on F.Cu, net V_IN
- added copper zone on B.Cu, net V_OUT
- added copper zone on F.Cu, net V_OUT

Commit message: done ish
Parts:
- added G***: LOGO, MRDT_Silkscreens:2_Nothing_3mm, F.Cu at (172.5, -25.9)
- moved D1 194.2 mm to (74.9, 12.7)
- moved C1 172.0 mm to (112.4, -18.4), turned to 90 degrees
- moved C9 147.1 mm to (129.5, -12.7), turned to 90 degrees
- moved U5 144.0 mm to (49.5, 156.2)
- moved C8 136.9 mm to (133.3, -12.7), turned to 90 degrees
- moved U7 129.2 mm to (34.3, 156.2)
- moved U3 128.1 mm to (66.0, 154.9)
- moved D2 125.2 mm to (82.5, 12.7)
- moved C5 119.7 mm to (144.8, -12.7), turned to 90 degrees
- moved C7 117.9 mm to (137.2, -12.7), turned to 90 degrees
- moved R22 116.5 mm to (111.8, 27.9)
- moved C4 116.4 mm to (148.6, -12.7), turned to 90 degrees
- moved C6 116.2 mm to (141.0, -12.7), turned to 90 degrees
- moved R29 113.2 mm to (158.8, 12.7)
- moved Conn9 112.6 mm to (160.0, -27.9)
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Connections:
- Conn1 pad 2: V_IN -> (no net)
Routing:
- net V_IN: track 211.2 -> 0.00 mm, vias 1 -> 0
- net (no net): track 0.00 -> 209.0 mm, vias 0 -> 1
- net Net-(R27-Pad2): track 1.49 -> 0.00 mm
- added copper zone on B.Cu, net GND
- added copper zone on F.Cu, net GND

Commit message: latest design before PDR
Parts:
- moved G*** 5.34 mm to (177.8, -25.7)
Connections:
- Conn1 pad 2: (no net) -> V_IN
Routing:
- net (no net): track 209.0 -> 0.00 mm, vias 1 -> 0
- net V_IN: track 0.00 -> 207.5 mm, vias 0 -> 1
- added copper zone on B.Cu, net PV
- added copper zone on F.Cu, net PV
- removed copper zone on B.Cu, net GND
- removed copper zone on F.Cu, net GND
Changed lines of the file:
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@@
     (thickness 1.6)
     (drawings 4)
-    (tracks 14)
+    (tracks 12)
     (zones 0)
     (modules 138)
@@
     (mod_text_width 0.15)
     (pad_size 5.08 5.08)
-    (pad_drill 4.104006)
+    (pad_drill 4.104005)
     (pad_to_mask_clearance 0.051)
     (solder_mask_min_width 0.25)
@@
   )
   (module MRDT_Silkscreens:2_Nothing_3mm (layer F.Cu)
-    (at 172.466 -25.908)
+    (at 177.8 -25.654)
     (fp_text reference G*** (at 2.6162 -3.5052) (layer F.SilkS) hide
       (effects (font (size 1.524 1.524) (thickness 0.3)))
@@
     (pad 1 thru_hole circle (at 3.95 -4.8 270) (size 5.08 5.08) (drill 4.104006) (layers *.Cu *.Mask)
       (net 4 GND))
-    (pad 2 thru_hole circle (at 11.85 -4.8 270) (size 5.08 5.08) (drill 4.104006) (layers *.Cu *.Mask))
+    (pad 2 thru_hole circle (at 11.85 -4.8 270) (size 5.08 5.08) (drill 4.104005) (layers *.Cu *.Mask)
+      (net 129 V_IN))
     (model "${MRDT_KICAD_LIBRARIES}/3D Files/MRDT_Connctors/Anderson_2_Vertcal_Side_by_Side.stp"
       (offset (xyz 15.87499976158142 6.984999895095826 0))
@@
   (gr_line (start 258.699 -30.861) (end 258.953 57.023) (layer F.SilkS) (width 0.12))
   (gr_line (start 36.703 -30.988) (end 258.699 -30.861) (layer F.SilkS) (width 0.12))
-  (gr_line (start 36.83 63.5) (end 36.703 -30.988) (layer F.SilkS) (width 0.12))
-  (segment (start 149.0205 22.606) (end 149.9065 22.606) (width 0.25) (layer F.Cu) (net 0))
-  (segment (start 150.5065 22.606) (end 149.9065 22.606) (width 0.25) (layer F.Cu) (net 0))
-  (segment (start 233.426 -29.464) (end 256.515778 -29.464) (width 2.54) (layer F.Cu) (net 0))
-  (via (at 251.46 16.51) (size 0.8) (drill 0.4) (layers F.Cu B.Cu) (net 0))
-  (segment (start 205.424 -29.464) (end 203.62 -27.66) (width 2.54) (layer F.Cu) (net 0))
-  (segment (start 233.450222 -29.464) (end 205.424 -29.464) (width 2.54) (layer F.Cu) (net 0))
-  (segment (start 205.424 -29.464) (end 203.62 -27.66) (width 2.54) (layer B.Cu) (net 0))
-  (segment (start 256.094 -29.464) (end 205.424 -29.464) (width 2.54) (layer B.Cu) (net 0))
-  (segment (start 256.54 15.24) (end 256.515778 -29.464) (width 2.54) (layer B.Cu) (net 0))
-  (segment (start 251.46 16.51) (end 252.73 15.24) (width 2.54) (layer B.Cu) (net 0))
-  (segment (start 252.73 15.24) (end 256.54 15.24) (width 2.54) (layer B.Cu) (net 0))
-  (segment (start 252.73 15.24) (end 251.46 16.51) (width 2.54) (layer F.Cu) (net 0))
-  (segment (start 256.515778 -29.464) (end 256.54 15.24) (width 2.54) (layer F.Cu) (net 0))
-  (segment (start 256.54 15.24) (end 252.73 15.24) (width 2.54) (layer F.Cu) (net 0))
+  (gr_line (start 36.83 57.15) (end 36.703 -30.988) (layer F.SilkS) (width 0.12))
+  (segment (start 233.426 -29.464) (end 256.515778 -29.464) (width 2.54) (layer F.Cu) (net 129))
+  (via (at 251.46 16.51) (size 0.8) (drill 0.4) (layers F.Cu B.Cu) (net 129))
+  (segment (start 205.424 -29.464) (end 203.62 -27.66) (width 2.54) (layer F.Cu) (net 129))
+  (segment (start 233.450222 -29.464) (end 205.424 -29.464) (width 2.54) (layer F.Cu) (net 129))
+  (segment (start 205.424 -29.464) (end 203.62 -27.66) (width 2.54) (layer B.Cu) (net 129))
+  (segment (start 256.094 -29.464) (end 205.424 -29.464) (width 2.54) (layer B.Cu) (net 129))
+  (segment (start 256.54 15.24) (end 256.515778 -29.464) (width 2.54) (layer B.Cu) (net 129))
+  (segment (start 251.46 16.51) (end 252.73 15.24) (width 2.54) (layer B.Cu) (net 129))
+  (segment (start 252.73 15.24) (end 256.54 15.24) (width 2.54) (layer B.Cu) (net 129))
+  (segment (start 252.73 15.24) (end 251.46 16.51) (width 2.54) (layer F.Cu) (net 129))
+  (segment (start 256.515778 -29.464) (end 256.54 15.24) (width 2.54) (layer F.Cu) (net 129))
+  (segment (start 256.54 15.24) (end 252.73 15.24) (width 2.54) (layer F.Cu) (net 129))
   (zone (net 129) (net_name V_IN) (layer F.Cu) (hatch edge 0.508)
-    (connect_pads (clearance 0.508))
+    (connect_pads yes (clearance 0.508))
     (min_thickness 0.254)
     (fill yes (arc_segments 32) (thermal_gap 0.508) (thermal_bridge_width 0.508))
     (polygon
       (pts
-        (xy 257.8862 56.9722) (xy 257.8862 11.9126) (xy 219.964 11.7475) (xy 219.71 56.8325) (xy 239.1918 57.0992)
+        (xy 257.81 56.515) (xy 257.81 12.7) (xy 219.71 12.7) (xy 219.71 37.465) (xy 222.862552 37.465)
+        (xy 222.907448 41.91) (xy 219.754896 41.91) (xy 219.71 56.515) (xy 239.1918 56.515)
       )
     )
   )
   (zone (net 129) (net_name V_IN) (layer B.Cu) (hatch edge 0.508)
-    (connect_pads (clearance 0.508))
+    (connect_pads yes (clearance 0.508))
     (min_thickness 0.254)
     (fill yes (arc_segments 32) (thermal_gap 0.508) (thermal_bridge_width 0.508))
     (polygon
       (pts
-        (xy 257.81 57.15) (xy 257.81 12.7) (xy 219.71 12.7) (xy 219.71 57.15)
+        (xy 257.81 56.515) (xy 257.81 12.7) (xy 219.71 12.7) (xy 219.71 37.465) (xy 222.885 37.465)
+        (xy 222.885 41.91) (xy 219.74175 41.91) (xy 219.71 56.515)
       )
     )
   )
   (zone (net 39) (net_name V_OUT) (layer F.Cu) (hatch edge 0.508)
-    (connect_pads (clearance 0.508))
+    (connect_pads yes (clearance 0.508))
     (min_thickness 0.254)
     (fill yes (arc_segments 32) (thermal_gap 0.508) (thermal_bridge_width 0.508))
     (polygon
       (pts
-        (xy 219.71 11.43) (xy 219.71 -29.21) (xy 255.27 -29.21) (xy 255.27 11.43)
+        (xy 219.71 10.795) (xy 219.71 -29.21) (xy 254.635 -29.845) (xy 254.635 10.795)
       )
     )
   )
   (zone (net 39) (net_name V_OUT) (layer B.Cu) (hatch edge 0.508)
-    (connect_pads (clearance 0.508))
+    (connect_pads yes (clearance 0.508))
     (min_thickness 0.254)
     (fill yes (arc_segments 32) (thermal_gap 0.508) (thermal_bridge_width 0.508))
     (polygon
       (pts
-        (xy 219.71 11.43) (xy 219.71 -29.21) (xy 255.27 -29.21) (xy 255.27 11.43) (xy 252.73 11.43)
+        (xy 219.71 10.795) (xy 219.71 -29.21) (xy 254.635 -29.21) (xy 254.635 10.795) (xy 252.73 10.795)
       )
     )
   )
-  (zone (net 4) (net_name GND) (layer B.Cu) (hatch edge 0.508)
-    (connect_pads (clearance 0.508))
+  (zone (net 3) (net_name PV) (layer F.Cu) (hatch edge 0.508)
+    (connect_pads yes (clearance 0.508))
     (min_thickness 0.254)
     (fill yes (arc_segments 32) (thermal_gap 0.508) (thermal_bridge_width 0.508))
     (polygon
       (pts
-        (xy 31.115 -38.1) (xy 259.08 -38.1) (xy 259.08 59.055) (xy 31.115 59.055) (xy 31.115 53.34)
+        (xy 201.316282 3.048) (xy 201.295 -17.145) (xy 216.535 -17.145) (xy 216.535 12.065) (xy 219.075 12.065)
+        (xy 219.075 20.32) (xy 219.075 37.592) (xy 201.316282 37.592)
       )
     )
   )
-  (zone (net 4) (net_name GND) (layer F.Cu) (hatch edge 0.508)
-    (connect_pads (clearance 0.508))
+  (zone (net 3) (net_name PV) (layer B.Cu) (hatch edge 0.508)
+    (connect_pads yes (clearance 0.508))
     (min_thickness 0.254)
     (fill yes (arc_segments 32) (thermal_gap 0.508) (thermal_bridge_width 0.508))
     (polygon
       (pts
-        (xy 259.08 -38.1) (xy 31.115 -38.1) (xy 31.115 59.055) (xy 259.08 59.055)
+        (xy 201.295 -17.145) (xy 216.535 -17.145) (xy 216.535 12.065) (xy 219.075 12.065) (xy 219.075 37.592)
+        (xy 201.295 37.592)
       )
     )

Commit message: PDR Ready
Parts:
- added G***: LOGO, MRDT_Silkscreens:0_MRDT_Logo_20mm, F.Cu at (64.8, -11.4)
- moved R54 9.27 mm to (50.2, -19.7)
- moved Q6 8.89 mm to (50.2, -15.9)
- moved R55 8.51 mm to (50.2, -10.8)
- moved Q7 8.38 mm to (50.2, -6.99)

Commit message: actual final before PDR :)
Parts:
- moved Q4 95.8 mm to (86.4, -10.8)
- moved R52 89.8 mm to (86.4, -14.6)
- moved B1 42.1 mm to (102.9, -1.27)
Changed lines of the file:
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@@
   )
   (module MRDT_Devices:BUZZER_SMI_1324_TW_5V_2_R (layer F.Cu)
-    (at 106.68 40.64)
+    (at 102.87 -1.27)
     (fp_text reference B1 (at 2.3 7.5) (layer F.SilkS)
       (effects (font (size 1 1) (thickness 0.15)))
@@
   )
   (module Package_TO_SOT_SMD:SOT-23 (layer F.Cu)
-    (at 180.34 7.62 270)
+    (at 86.36 -10.795 270)
     (descr "SOT-23, Standard")
     (tags SOT-23)
@@
   )
   (module Resistor_SMD:R_0603_1608Metric_Pad1.05x0.95mm_HandSolder (layer F.Cu)
-    (at 173.482 6.985)
+    (at 86.36 -14.605)
     (descr "Resistor SMD 0603 (1608 Metric), square (rectangular) end terminal, IPC_7351 nominal with elongated pad for handsoldering. (Body size source: http://www.tortai-tech.com/upload/download/2011102023233369053.pdf), generated with kicad-footprint-generator")
     (tags "resistor handsolder")

Commit message: haha it wasnt ready till now
Parts:
- added U11: TM4C129E_Launchpad, MRDT_Shields:TM4C129E_Launchpad_FULL_SMD_TOP, F.Cu at (67.7, 45.5)
- F1: footprint Fuse:Fuse_0603_1608Metric_Pad1.05x0.95mm_HandSolder -> Fuse:Fuse_2920_7451Metric
- moved F1 20.6 mm to (181.0, 1.27)
Connections:
- Conn1 pad 2: V_IN -> (no net)
- R15 pad 2: Net-(R15-Pad2) -> CELL8_SENSE
- R17 pad 2: Net-(R17-Pad2) -> CELL7_SENSE
- R19 pad 2: Net-(R19-Pad2) -> CELL6_SENSE
- R21 pad 2: Net-(R21-Pad2) -> CELL5_SENSE
- R23 pad 2: Net-(R23-Pad2) -> CELL4_SENSE
- R25 pad 2: Net-(R25-Pad2) -> CELL3_SENSE
- R27 pad 2: Net-(R27-Pad2) -> CELL2_SENSE
- U2 pad 3: Net-(R15-Pad2) -> CELL8_SENSE
- U2 pad 4: +5V -> LOGIC_PWR
- U3 pad 3: Net-(R17-Pad2) -> CELL7_SENSE
- U3 pad 4: +5V -> LOGIC_PWR
- U4 pad 3: Net-(R19-Pad2) -> CELL6_SENSE
- U4 pad 4: +5V -> LOGIC_PWR
- U5 pad 3: Net-(R21-Pad2) -> CELL5_SENSE
- U5 pad 4: +5V -> LOGIC_PWR
- U6 pad 3: Net-(R23-Pad2) -> CELL4_SENSE
- U6 pad 4: +5V -> Net-(U6-Pad4)
- U7 pad 3: Net-(R25-Pad2) -> CELL3_SENSE
- U7 pad 4: +5V -> Net-(U7-Pad4)
- U8 pad 3: Net-(R27-Pad2) -> CELL2_SENSE
- U8 pad 4: +5V -> Net-(U8-Pad4)
Routing:
- net V_IN: track 207.5 -> 0.00 mm, vias 1 -> 0
- net (no net): track 0.00 -> 207.5 mm, vias 0 -> 1
