File: BMS_Hardware/_autosave-2020_BMSBOARD.kicad_pcb (KiCad board)
At the start: 2 copper layers, 170.2 x 76.2 mm, 133 parts, among them Q1 2N7002, Q2 Q_NMOS_GDS, Q3 Device_Q_NMOS_GDS, Q4 2N7002PW, Q5 2N7002PW, Q7 2N7002PW, SW1 Relay_SPST-MRDT_Switches, U1 LT1910, U10 OKI, U12 OKI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

Commit message: don't be dan
Parts:
- C2, C3, C4, C5, C6, C7, C8: value C -> 1u
- Conn2: footprint MRDT_Connectors:MOLEX_SL_02_Vertical -> MRDT_Connectors:MOLEX_SL_04_Vertical; moved to F.Cu
- D10, D11, D12, D13, D14, D15, D16, D23: value 3.3V -> 3V3
- D9: value D_Zener -> 3V3
- R53, R55: value 100K -> 10K
- moved Conn2 6.48 mm to (137.7, -6.73), turned to 0 degrees
Connections:
- Conn1 pad 2: V_IN -> (no net)
- Conn2 pad 1: Net-(Conn2-Pad1) -> +5V
- Conn2 pad 2: Net-(Conn2-Pad2) -> GND
- Conn3 pad 1: Net-(Conn2-Pad2) -> Net-(Conn2-Pad4)
- R30 pad 1: Net-(Conn2-Pad1) -> Net-(Conn2-Pad3)
- U1 pad 4: Net-(Conn2-Pad1) -> Net-(Conn2-Pad3)
- U6 pad NC: FAN_PWR_IND -> Net-(U6-PadNC)
- U6 pad PA0: FAN_CTL_1 -> Net-(U6-PadPA0)
- U6 pad PF2: Net-(U6-PadPF2) -> FAN_PWR_IND
- U6 pad PK0: Net-(U6-PadPK0) -> FAN_CTL_1
Routing:
- net V_IN: track 216.9 -> 0.00 mm
- net (no net): track 0.00 -> 216.9 mm
- net Net-(Conn2-Pad3): track 0.00 -> 64.6 mm, vias 0 -> 2
- net Net-(Conn2-Pad1): track 64.6 -> 0.00 mm, vias 2 -> 0
- net Net-(R22-Pad2): track 32.5 -> 16.5 mm
- net Net-(Conn2-Pad4): track 0.00 -> 14.3 mm, vias 0 -> 2
- net Net-(Conn2-Pad2): track 14.3 -> 0.00 mm, vias 2 -> 0
- net Net-(R18-Pad2): track 50.5 -> 43.3 mm
- net Net-(R20-Pad2): track 12.8 -> 5.92 mm
