File: Hardware/BMS_2021_Rev1/_autosave-CURRENT_SENSE.sch (KiCad schematic (older format))
At the start: 8 parts

Commit message: stuff added
-cellFilter IC and R values added
-MOSFET values added
-extra TIVA headers added
-currentSense R values labeled properly
-things are actually connected together this time
Parts:
- removed R? (x2): 5mΩ, symbol Device:R
- added J? (x3): Test_Point, symbol MRDT_Connectors:Test_Point
- added R? (x2): 50mΩ, symbol Device:R
- R?: value 5mΩ -> 50mΩ
- U?: value INA281 -> INA281A
Connections:
- wire segments 33 -> 37
Other:
- note removed: "<-- 50 mOhm\n"
- note removed: "new IC: take voltage across shunt, done and dusted\n"
Changed lines of the file:
@@
 Text HLabel 3550 850  2    50   Input ~ 0
 V_in
-$Comp
-L Device:R R?
-U 1 1 5F83ACC9
-P 1800 850
-F 0 "R?" V 1700 850 50  0000 C CNN
-F 1 "5mΩ" V 1800 850 39  0000 C CNN
-F 2 "" V 1730 850 50  0001 C CNN
-F 3 "~" H 1800 850 50  0001 C CNN
-	1    1800 850
-	0    1    1    0
-$EndComp
-$Comp
-L Device:R R?
-U 1 1 5F83B3DE
-P 2200 850
-F 0 "R?" V 2100 850 50  0000 C CNN
-F 1 "5mΩ" V 2200 850 39  0000 C CNN
-F 2 "" V 2130 850 50  0001 C CNN
-F 3 "~" H 2200 850 50  0001 C CNN
-	1    2200 850
-	0    1    1    0
-$EndComp
 Wire Wire Line
 	2350 850  2450 850
@@
 Connection ~ 2850 850
 Wire Wire Line
-	2850 850  3550 850
+	2850 850  2925 850
 $Comp
 L Device:R R?
@@
 P 2600 850
 F 0 "R?" V 2500 850 50  0000 C CNN
-F 1 "5mΩ" V 2600 850 39  0000 C CNN
+F 1 "50mΩ" V 2600 850 39  0000 C CNN
 F 2 "" V 2530 850 50  0001 C CNN
-F 3 "~" H 2600 850 50  0001 C CNN
+F 3 "https://www.digikey.com/en/products/detail/riedon/PF2472-0R05J1/2447851" H 2600 850 50  0001 C CNN
 	1    2600 850
 	0    1    1    0
@@
 U 1 1 5F86B7DF
 P 2200 1600
-F 0 "U?" V 2254 1944 50  0000 L CNN
-F 1 "INA281" V 2345 1944 50  0000 L CNN
+F 0 "U?" V 2325 1725 50  0000 L CNN
+F 1 "INA281A" V 2425 1725 50  0000 L CNN
 F 2 "" H 2450 1800 50  0001 C CNN
 F 3 "https://www.ti.com/product/INA281" H 2450 1800 50  0001 C CNN
@@
 Text HLabel 2350 2400 2    50   Output ~ 0
 pack_i_sense
-Text Notes 4100 900  0    50   ~ 10
-<-- 50 mOhm\n
-Text Notes 4250 1875 0    50   ~ 10
-new IC: take voltage across shunt, done and dusted\n
 Wire Wire Line
 	900  850  1550 850
@@
 Wire Wire Line
 	2200 2400 2350 2400
+$Comp
+L MRDT_Connectors:Test_Point J?
+U 1 1 5FA757F5
+P 2925 725
+F 0 "J?" H 3003 870 60  0000 L CNN
+F 1 "Test_Point" H 3003 764 60  0000 L CNN
+F 2 "" H 2925 675 60  0001 C CNN
+F 3 "" H 2925 675 60  0001 C CNN
+	1    2925 725
+	1    0    0    -1
+$EndComp
+Wire Wire Line
+	2925 725  2925 850
+Connection ~ 2925 850
+Wire Wire Line
+	2925 850  3550 850
+$Comp
+L MRDT_Connectors:Test_Point J?
+U 1 1 5FA7660C
+P 1475 725
+F 0 "J?" H 1325 875 60  0000 L CNN
+F 1 "Test_Point" H 1000 775 60  0000 L CNN
+F 2 "" H 1475 675 60  0001 C CNN
+F 3 "" H 1475 675 60  0001 C CNN
+	1    1475 725
+	1    0    0    -1
+$EndComp
+Wire Wire Line
+	1475 725  1475 850
+$Comp
+L MRDT_Connectors:Test_Point J?
+U 1 1 5FAAFB1B
+P 2075 2400
+F 0 "J?" V 2175 2500 60  0000 L CNN
+F 1 "Test_Point" V 1975 2325 60  0000 L CNN
+F 2 "" H 2075 2350 60  0001 C CNN
+F 3 "" H 2075 2350 60  0001 C CNN
+	1    2075 2400
+	0    -1   -1   0
+$EndComp
+Wire Wire Line
+	2075 2400 2200 2400
+$Comp
+L Device:R R?
+U 1 1 5FAB1180
+P 2200 850
+F 0 "R?" V 2100 850 50  0000 C CNN
+F 1 "50mΩ" V 2200 850 39  0000 C CNN
+F 2 "" V 2130 850 50  0001 C CNN
+F 3 "https://www.digikey.com/en/products/detail/riedon/PF2472-0R05J1/2447851" H 2200 850 50  0001 C CNN
+	1    2200 850
+	0    1    1    0
+$EndComp
+$Comp
+L Device:R R?
+U 1 1 5FAB1A87
+P 1800 850
+F 0 "R?" V 1700 850 50  0000 C CNN
+F 1 "50mΩ" V 1800 850 39  0000 C CNN
+F 2 "" V 1730 850 50  0001 C CNN
+F 3 "https://www.digikey.com/en/products/detail/riedon/PF2472-0R05J1/2447851" H 1800 850 50  0001 C CNN
+	1    1800 850
+	0    1    1    0
+$EndComp
 $EndSCHEMATC

Commit message: added libraries to docs folder
Connections:
- wire segments 37 -> 38
Other:
- moved on the sheet: Q?, R?
Changed lines of the file:
@@
 L Device:R R?
 U 1 1 5F8362F1
-P 1975 5725
-F 0 "R?" V 1885 5725 50  0000 C CNN
-F 1 "27Ω" V 1975 5725 39  0000 C CNN
-F 2 "" V 1905 5725 50  0001 C CNN
-F 3 "~" H 1975 5725 50  0001 C CNN
-	1    1975 5725
+P 9350 5400
+F 0 "R?" V 9260 5400 50  0000 C CNN
+F 1 "27Ω" V 9350 5400 39  0000 C CNN
+F 2 "" V 9280 5400 50  0001 C CNN
+F 3 "~" H 9350 5400 50  0001 C CNN
+	1    9350 5400
 	0    1    1    0
 $EndComp
@@
 L Device:R R?
 U 1 1 5F83721F
-P 2675 5725
-F 0 "R?" V 2585 5725 50  0000 C CNN
-F 1 "27Ω" V 2675 5725 39  0000 C CNN
-F 2 "" V 2605 5725 50  0001 C CNN
-F 3 "~" H 2675 5725 50  0001 C CNN
-	1    2675 5725
-	0    1    1    0
-$EndComp
-Wire Wire Line
-	2825 5725 2975 5725
-Wire Wire Line
-	1675 5725 1825 5725
-Wire Wire Line
-	1675 5425 1675 5725
-Wire Wire Line
-	2125 5725 2225 5725
-Wire Wire Line
-	2425 5725 2525 5725
+P 10050 5400
+F 0 "R?" V 9960 5400 50  0000 C CNN
+F 1 "27Ω" V 10050 5400 39  0000 C CNN
+F 2 "" V 9980 5400 50  0001 C CNN
+F 3 "~" H 10050 5400 50  0001 C CNN
+	1    10050 5400
+	0    1    1    0
+$EndComp
+Wire Wire Line
+	10200 5400 10350 5400
+Wire Wire Line
+	9050 5400 9200 5400
+Wire Wire Line
+	9050 5100 9050 5400
+Wire Wire Line
+	9500 5400 9600 5400
+Wire Wire Line
+	9800 5400 9900 5400
 Wire Wire Line
 	2500 1600 2700 1600
@@
 $EndComp
 Wire Wire Line
-	2225 5725 2225 5875
-Wire Wire Line
-	2425 5725 2425 5975
-Connection ~ 2225 5875
-Wire Wire Line
-	2225 5875 2225 5975
-Wire Wire Line
-	975  3175 975  4175
-Wire Wire Line
-	1675 5875 2225 5875
+	9600 5400 9600 5550
+Wire Wire Line
+	9800 5400 9800 5650
+Connection ~ 9600 5550
+Wire Wire Line
+	9600 5550 9600 5650
+Wire Wire Line
+	8350 2850 8350 3850
+Wire Wire Line
+	9050 5550 9600 5550
 $Comp
 L Device:Q_NMOS_DGS Q?
 U 1 1 5F852FE1
-P 1525 4175
-F 0 "Q?" H 1729 4221 50  0000 L CNN
-F 1 "Q_NMOS_DGS" H 1729 4130 50  0000 L CNN
-F 2 "" H 1725 4275 50  0001 C CNN
-F 3 "~" H 1525 4175 50  0001 C CNN
-	1    1525 4175
-	1    0    0    -1
-$EndComp
-Wire Wire Line
-	1625 3875 1625 3975
-Wire Wire Line
-	975  4175 1325 4175
-Wire Wire Line
-	1625 4375 1625 4525
+P 8900 3850
+F 0 "Q?" H 9104 3896 50  0000 L CNN
+F 1 "Q_NMOS_DGS" H 9104 3805 50  0000 L CNN
+F 2 "" H 9100 3950 50  0001 C CNN
+F 3 "~" H 8900 3850 50  0001 C CNN
+	1    8900 3850
+	1    0    0    -1
+$EndComp
+Wire Wire Line
+	9000 3550 9000 3650
+Wire Wire Line
+	8350 3850 8700 3850
+Wire Wire Line
+	9000 4050 9000 4200
 $Comp
 L Device:R R?
 U 1 1 5F85658D
-P 1625 4775
-F 0 "R?" H 1555 4775 50  0000 R CNN
-F 1 "330Ω" V 1625 4855 39  0000 R CNN
-F 2 "" V 1555 4775 50  0001 C CNN
-F 3 "~" H 1625 4775 50  0001 C CNN
-	1    1625 4775
+P 9000 4450
+F 0 "R?" H 8930 4450 50  0000 R CNN
+F 1 "330Ω" V 9000 4530 39  0000 R CNN
+F 2 "" V 8930 4450 50  0001 C CNN
+F 3 "~" H 9000 4450 50  0001 C CNN
+	1    9000 4450
 	-1   0    0    1
 $EndComp
 Wire Wire Line
-	1625 4925 1625 5025
+	9000 4600 9000 4700
 $Comp
 L power:GND #PWR?
 U 1 1 5F859B0F
-P 1625 5025
-F 0 "#PWR?" H 1625 4775 50  0001 C CNN
-F 1 "GND" H 1630 4852 50  0000 C CNN
-F 2 "" H 1625 5025 50  0001 C CNN
-F 3 "" H 1625 5025 50  0001 C CNN
-	1    1625 5025
+P 9000 4700
+F 0 "#PWR?" H 9000 4450 50  0001 C CNN
+F 1 "GND" H 9005 4527 50  0000 C CNN
+F 2 "" H 9000 4700 50  0001 C CNN
+F 3 "" H 9000 4700 50  0001 C CNN
+	1    9000 4700
 	1    0    0    -1
 $EndComp
@@
 	1750 1600 1900 1600
 Wire Wire Line
-	1625 4525 1950 4525
-Connection ~ 1625 4525
-Wire Wire Line
-	1625 4525 1625 4625
+	9000 4200 9325 4200
+Connection ~ 9000 4200
+Wire Wire Line
+	9000 4200 9000 4300
 Text HLabel 2350 2400 2    50   Output ~ 0
 pack_i_sense
 Wire Wire Line
-	900  850  1550 850
-Wire Wire Line
 	1550 850  1550 1225
 Wire Wire Line
@@
 Wire Wire Line
 	2100 1225 2100 1400
-Connection ~ 1550 850
 Wire Wire Line
 	1550 850  1650 850
@@
 	1    0    0    -1
 $EndComp
-Wire Wire Line
-	1475 725  1475 850
 $Comp
 L MRDT_Connectors:Test_Point J?
@@
 	0    1    1    0
 $EndComp
+Wire Wire Line
+	1550 850  1475 850
+Connection ~ 1550 850
+Wire Wire Line
+	1475 850  1475 725
+Connection ~ 1475 850
+Wire Wire Line
+	1475 850  900  850
 $EndSCHEMATC
