File: Hardware/BMS_2021_Rev1/_autosave-BMS_2021_Rev1.kicad_pcb (KiCad board)
At the start: 2 copper layers, 120 parts, among them J2 Test_Point, J4 Test_Point, J5 Test_Point, Q1 2N7002PW, Q2 IRLB3034PBF, Q3 IRLB3034PBF, Q4 2N7000, Q5 2N7002PW, SW1 Relay_SPST, U1 TM4C129E_Launchpad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

Commit message: estop circuit finished being placed, back Vin/Vout polygon made
Need to add vias to connect the front and back polygons
Parts:
- moved D17 164.4 mm to (207.0, 59.7)
- moved Q3 163.6 mm to (207.0, 48.3), turned to 270 degrees
- moved Q2 157.4 mm to (213.4, 55.9), turned to 90 degrees
- moved C11 13.3 mm to (165.1, 83.8), turned to 0 degrees
- moved U7 9.25 mm to (158.8, 78.7), turned to 90 degrees
- moved R41 8.05 mm to (176.5, 78.7), turned to 270 degrees
- moved U1 6.48 mm to (147.3, 49.5)
- moved R39 6.21 mm to (170.2, 78.7), turned to 270 degrees
- moved R40 2.48 mm to (176.5, 74.9), turned to 270 degrees
- moved R38 0.66 mm to (170.2, 74.9), turned to 270 degrees

Commit message: Q2,3 footprint updated, via stitched V_in, TIVA moved
-need to update schematic symbols Q2,3
-double check TIVA orientation
Parts:
- moved U1 95.5 mm to (63.5, 95.2), turned to 0 degrees
Routing:
- net /V_in: track 115.6 -> 115.9 mm, vias 1 -> 189
- net /PV: vias 1 -> 0
- net /ESTOP/V_out: vias 0 -> 6
- added copper zone on B.Cu, net /ESTOP/V_out
- added copper zone on B.Cu, net /V_in
