File: Hardware/2023rev2.0/2023rev2.0.kicad_pcb (KiCad board)
At the start: 2 copper layers, 88 parts, among them J1 Conn_01x03, J2 Conn_01x09, J3 Conn_01x09, J4 Conn_01x04, Q1 Q_NMOS_DGS, SW1 SW_SPDT, U1 Teensy4.1_DEV-16771, U2 Opamp_Dual, U3 Opamp_Dual, U4 Opamp_Dual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

Commit message: Start Placing Mounting Holes
Parts:
- removed C4: 22uF, Capacitor_THT:CP_Radial_D5.0mm_P2.50mm
- removed C5: 1uF, Capacitor_THT:CP_Radial_D5.0mm_P2.50mm
- removed C6: 10uF, Capacitor_THT:CP_Radial_D5.0mm_P2.50mm
- added H1: MountingHole, MRDT_Drill_Holes:4_40_Hole, F.Cu at (260.9, 126.8)
- added H2: MountingHole, MRDT_Drill_Holes:4_40_Hole, F.Cu at (260.9, 117.6)
- added H3: MountingHole, MRDT_Drill_Holes:4_40_Hole, F.Cu at (318.0, 203.5)
- added H4: MountingHole, MRDT_Drill_Holes:4_40_Hole, F.Cu at (52.1, 206.2)
- added H5: MountingHole, MRDT_Drill_Holes:4_40_Hole, F.Cu at (251.7, 126.8)
- added H6: MountingHole, MRDT_Drill_Holes:4_40_Hole, F.Cu at (251.7, 117.6)
- added U6: INA195, Package_TO_SOT_SMD:SOT-23-6, F.Cu at (151.1, 104.6)
- moved V2 308.8 mm to (297.9, 186.9)
- moved J1 166.9 mm to (260.6, 46.0)
- moved J4 143.9 mm to (238.0, 46.2)
- moved BZ1 136.0 mm to (98.9, 161.3)
- moved R3 121.0 mm to (185.2, 152.0)
- moved R9 121.0 mm to (189.6, 152.0)
- moved C2 121.0 mm to (169.7, 157.2)
- moved D10 121.0 mm to (186.1, 147.0)
- moved D11 121.0 mm to (160.3, 171.3)
- moved D15 121.0 mm to (160.3, 168.7)
- moved D16 121.0 mm to (190.4, 144.4)
- moved D17 121.0 mm to (181.7, 149.5)
- moved D18 121.0 mm to (180.9, 153.3)
- moved D19 121.0 mm to (186.1, 144.4)
- moved D20 121.0 mm to (172.8, 161.8)
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- renumbered R42 to R41, U9 to U8
Connections:
- U1 pad 11: Net-(U1-Pad11) -> unconnected-(U1-Pad11)
Other:
- board outline added: 279.4 x 181.4 mm

Commit message: Placed Mounting Holes
Parts:
- moved H5 204.5 mm to (52.1, 82.5)
- moved R36 95.5 mm to (156.1, 68.8)
- moved R33 81.9 mm to (154.8, 79.6)
- moved H1 80.4 mm to (255.9, 207.0)
- moved R35 78.0 mm to (160.6, 77.9)
- moved R18 78.0 mm to (175.8, 70.9), turned to 90 degrees
- moved R16 74.2 mm to (161.0, 83.3), turned to 90 degrees
- moved R32 74.2 mm to (155.1, 83.3), turned to -90 degrees
- moved R20 72.8 mm to (162.4, 68.3), turned to 90 degrees
- moved H2 69.8 mm to (321.3, 82.5)
- moved R17 64.0 mm to (169.5, 77.3)
- moved R31 62.0 mm to (167.9, 90.9)
- moved R13 56.0 mm to (172.0, 91.2), turned to 180 degrees
- moved R30 48.8 mm to (177.8, 89.3)
- moved R19 43.7 mm to (162.6, 72.3), turned to -90 degrees
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