File: Hardware/2023Rev2/2023Rev2.kicad_pcb (KiCad board)
At the start: 2 copper layers, 90 parts, among them J2 Conn_01x03, J3 Conn_01x03, J4 Conn_01x02, J5 Conn_01x09, J6 Conn_01x09, J7 RJ45_LED_Shielded, J9 Conn_01x04, Q2 Q_NMOS_DGS, Q3 Q_NMOS_DGS, Q4 Q_NMOS_DGS, Q5 Q_NMOS_GDS, U10 LT1910, U11 TSR_1-2450, U2 Opamp_Dual, U3 Teensy4.1_DEV-16771, U4 Opamp_Dual, U5 Opamp_Dual, U6 Opamp_Dual, U7 ACS758xCB-200B-PFF, U8 BMS_Logic_Switch, U9 OKI

Commit message: Placing Connectors on Schematic
Decided to put smaller components on back side.
Parts:
- moved R4 219.3 mm to (36.9, 137.2)
- moved R42 204.4 mm to (49.8, 99.7), turned to 90 degrees
- moved R13 197.5 mm to (77.3, 87.2)
- moved R16 197.5 mm to (60.7, 107.5)
- moved R24 197.5 mm to (60.7, 110.0)
- moved R26 197.5 mm to (77.3, 89.7)
- moved R27 197.5 mm to (69.8, 96.4)
- moved R34 197.5 mm to (77.3, 92.2)
- moved R36 197.5 mm to (61.1, 102.5)
- moved R41 197.5 mm to (60.7, 105.0)
- moved R46 197.5 mm to (69.8, 98.9)
- moved C2 197.5 mm to (65.5, 101.4)
- moved R18 197.5 mm to (65.4, 96.4)
- moved R30 197.5 mm to (65.4, 98.9)
- moved R33 197.5 mm to (65.5, 103.9)
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
Commit message: Layout of major components except opamps
Parts:
- added H7: MountingHole, MRDT_Drill_Holes:4_40_Hole, F.Cu at (178.1, 66.4)
- added H7: MountingHole, MRDT_Drill_Holes:4_40_Hole, F.Cu at (178.1, 104.4)
- R18, R2, R20, R3, R30, R37, R4, R40, R41, R42, R5, R7, R8, U2, U4, U5, U6: moved to B.Cu
- moved R4 149.1 mm to (172.5, 75.2), turned to -90 degrees
- moved U2 140.3 mm to (166.4, 74.9), turned to 180 degrees
- moved R2 128.7 mm to (173.5, 78.0)
- moved U4 115.3 mm to (152.4, 74.9), turned to 180 degrees
- moved R18 107.7 mm to (158.0, 41.4), turned to -90 degrees
- moved U5 106.5 mm to (139.7, 74.9), turned to 180 degrees
- moved H3 103.3 mm to (195.9, 74.9)
- moved U11 96.0 mm to (96.4, 76.6)
- moved R30 95.3 mm to (144.8, 46.2), turned to -90 degrees
- moved R5 95.0 mm to (160.3, 76.5), turned to 90 degrees
- moved R7 90.7 mm to (170.9, 74.2), turned to -90 degrees
- moved H7 81.0 mm to (100.8, 66.4)
- moved U6 78.6 mm to (127.0, 74.9), turned to 180 degrees
- moved H2 78.2 mm to (205.2, 74.9)
- moved R3 75.9 mm to (161.8, 75.9), turned to -90 degrees
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Routing:
- net cell7: track 0.00 -> 9.95 mm
- net Net-(R8-Pad2): track 0.00 -> 9.12 mm
- net Net-(R4-Pad2): track 0.00 -> 8.97 mm
- net cell8: track 0.00 -> 8.00 mm
- net cell5: track 0.00 -> 8.00 mm
- net cell4: track 0.00 -> 8.00 mm
- net cell3: track 0.00 -> 8.00 mm
- net cell2: track 0.00 -> 8.00 mm
- net cell1: track 0.00 -> 8.00 mm
- net call6: track 0.00 -> 8.00 mm
- net Net-(R37-Pad2): track 0.00 -> 2.62 mm
- net Net-(R6-Pad1): track 0.00 -> 2.20 mm
- net Net-(R2-Pad1): track 0.00 -> 2.01 mm
Other:
- board outline added: 101.6 x 97.8 mm

Commit message: Completed Layout
Parts:
- removed D8: Pack, LED_SMD:LED_0603_1608Metric_Pad1.05x0.95mm_HandSolder
- removed H2, H4, H5: MountingHole, MRDT_Drill_Holes:4_40_Hole_Corner
- removed H6, H7 (x3): MountingHole, MRDT_Drill_Holes:4_40_Hole
- added C7: 22uF, Capacitor_THT:CP_Radial_D5.0mm_P2.00mm, F.Cu at (75.9, 38.1)
- added C8: 1uF, Capacitor_SMD:C_0603_1608Metric_Pad1.08x0.95mm_HandSolder, F.Cu at (87.6, 27.9)
- added C9: 10uF, Capacitor_SMD:C_0603_1608Metric_Pad1.08x0.95mm_HandSolder, F.Cu at (88.4, 33.0)
- added D9: LED, LED_SMD:LED_0603_1608Metric_Pad1.05x0.95mm_HandSolder, F.Cu at (132.1, 79.0)
- added R47: 75, Resistor_SMD:R_0603_1608Metric_Pad0.98x0.95mm_HandSolder, F.Cu at (132.1, 84.3)
- added R48: 75, Resistor_SMD:R_0603_1608Metric_Pad0.98x0.95mm_HandSolder, F.Cu at (132.1, 87.8)
- added R50: 75, Resistor_SMD:R_0603_1608Metric_Pad0.98x0.95mm_HandSolder, F.Cu at (132.1, 80.8)
- C2: footprint Capacitor_SMD:C_0603_1608Metric_Pad1.08x0.95mm_HandSolder -> Capacitor_THT:CP_Radial_D5.0mm_P2.00mm
- C3: footprint Capacitor_SMD:C_0603_1608Metric_Pad1.08x0.95mm_HandSolder -> Capacitor_SMD:C_1210_3225Metric_Pad1.33x2.70mm_HandSolder
- D2: value Fan -> LED
- D3: value Buzzer -> LED
- H3: footprint MRDT_Drill_Holes:4_40_Hole_Corner -> MRDT_Drill_Holes:4_40_Hole
- R18, R2, R20, R3, R30, R37, R4, R40, R41, R42, R5, R7, R8, U2, U4, U5, U6: moved to F.Cu
- U3: footprint MRDT_Shields:Teensy_4_1 -> MRDT_Shields:Teensy_4_1_Ethernet
- moved R14 165.9 mm to (154.2, 62.4), turned to 90 degrees
- moved R31 165.2 mm to (158.2, 53.1), turned to 180 degrees
- moved R22 163.4 mm to (151.3, 58.7), turned to 180 degrees
- moved Q2 155.8 mm to (134.4, 65.0)
- moved R9 153.9 mm to (155.7, 70.8), turned to -90 degrees
- moved R39 147.9 mm to (154.2, 45.7), turned to 90 degrees
- moved D6 147.3 mm to (132.1, 68.3), turned to 180 degrees
- moved R10 144.9 mm to (147.8, 67.1), turned to 180 degrees
- moved R38 139.9 mm to (154.7, 50.3), turned to 180 degrees
- moved R23 139.7 mm to (158.2, 58.7), turned to 180 degrees
- moved D2 139.2 mm to (132.1, 82.5), turned to 180 degrees
- moved R21 131.9 mm to (147.8, 58.7), turned to 180 degrees
- moved D4 129.5 mm to (132.1, 89.7), turned to 180 degrees
- moved R12 129.0 mm to (158.2, 67.1), turned to 180 degrees
- moved C3 127.4 mm to (113.8, 53.3)
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Connections:
- C2 pad 1: Net-(C2-Pad1) -> PackLogic
- C3 pad 1: Net-(C3-Pad1) -> Net-(F2-Pad1)
- D2 pad 1: Net-(D2-Pad1) -> GND
- D2 pad 2: Net-(D2-Pad2) -> Net-(R47-Pad1)
- D3 pad 1: Net-(D3-Pad1) -> GND
- D3 pad 2: Net-(BZ2-Pad2) -> Net-(R48-Pad1)
- F2 pad 1: Net-(C3-Pad1) -> Net-(F2-Pad1)
- J4 pad 1: Net-(D2-Pad2) -> Net-(J4-Pad1)
- J6 pad 1: cell8 -> GND
- J6 pad 2: cell7 -> cell1
- J6 pad 3: call6 -> cell2
- J6 pad 4: cell5 -> cell3
- J6 pad 6: cell3 -> cell5
- J6 pad 7: cell2 -> call6
- J6 pad 8: cell1 -> cell7
- J6 pad 9: GND -> cell8
- Q2 pad 3: Net-(D2-Pad2) -> Net-(J4-Pad1)
- Q5 pad 1: Net-(C3-Pad1) -> Net-(Q5-Pad1)
- Q5 pad 2: Net-(C3-Pad1) -> Net-(F2-Pad1)
- U10 pad 5: Net-(C3-Pad1) -> Net-(Q5-Pad1)
- U10 pad 6: Net-(C3-Pad1) -> Net-(F2-Pad1)
- U10 pad 8: Net-(C3-Pad1) -> Net-(F2-Pad1)
- U11 pad 1: Net-(C2-Pad1) -> PackLogic
- U2 pad 8: PACK_OUT -> PackLogic
- U4 pad 8: PACK_OUT -> PackLogic
- U5 pad 8: PACK_OUT -> PackLogic
- U6 pad 8: PACK_OUT -> PackLogic
- U7 pad 5: Net-(C3-Pad1) -> Net-(F2-Pad1)
- U8 pad 3: Net-(C2-Pad1) -> PackLogic
- U9 pad 1: Net-(C2-Pad1) -> PackLogic
Routing:
- net PackLogic: track 0.00 -> 212.7 mm, vias 0 -> 7
- net CURRENT_SENSE: track 0.00 -> 201.0 mm, vias 0 -> 2
- net +3.3V: track 0.00 -> 157.7 mm
- net +5V: track 0.00 -> 149.9 mm, vias 0 -> 7
- net ERR_LED: track 0.00 -> 112.8 mm
- net PACK_OUT: track 0.00 -> 111.9 mm, vias 0 -> 39
- net Cell7-SENSE: track 0.00 -> 86.5 mm, vias 0 -> 3
- net Cell5-SENSE: track 0.00 -> 72.8 mm, vias 0 -> 3
- net Cell8-SENSE: track 0.00 -> 71.4 mm, vias 0 -> 2
- net Net-(Q3-Pad1): track 0.00 -> 70.5 mm
- net Net-(Q2-Pad1): track 0.00 -> 69.3 mm, vias 0 -> 7
- net Net-(Q4-Pad3): track 0.00 -> 64.6 mm, vias 0 -> 2
- net Cell3-SENSE: track 0.00 -> 60.5 mm, vias 0 -> 3
- net Cell6-SENSE: track 0.00 -> 58.3 mm, vias 0 -> 2
- net LOGIC_SWITCH: track 0.00 -> 50.4 mm, vias 0 -> 3
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- added copper zone on B.Cu, net GND
- added copper zone on F.Cu, net GND
- added copper zone on B.Cu, net Net-(Conn2-Pad2)
- added copper zone on F.Cu, net Net-(Conn2-Pad2)
- added copper zone on B.Cu, net Net-(F2-Pad1)
- added copper zone on F.Cu, net Net-(F2-Pad1)
- added copper zone on B.Cu, net PACK_OUT
- added copper zone on F.Cu, net PACK_OUT
Other:
- board size 101.6 x 97.8 mm -> 102.6 x 96.5 mm
- board text added: "+ D -"
- board text added: "- +"
- board text added: "3.3V"
- board text added: "5V"
- board text added: "Buzzer"
- board text added: "ESTOP"
- board text added: "Error"
- board text added: "FAN"
- board text added: "Fan"
- board text added: "GND C1 ^ C8"
- board text added: "LCD"
- board text added: "Logic"
- board text added: "Logic Switch"
- board text added: "TEMP"
- board text added: "V Out"
